File: eagle/nucleo-io-board/io-board-a-4.brd (EAGLE design)
At the start: 100 x 80 mm, 52 parts, among them IC1 74166N, IC3 74HCT595N, IC4 74166N, IC5 74HCT595N, IC6 LM324N, IC7 PCA82C250, IC9 LM324N, J1 RJ45-JACKRJ45-PULSE-E5J00, J2 RJ45-JACKRJ45-PULSE-E5J00, J3 DCJ0202

Commit message: More work on the nucleo io board.
Parts:
- added IC10: LM2574N-5.0, linear:DIL08
- added JP11: (no value), jumper:JP3Q
- added JP12: (no value), pinhead:2X05
- added JP13, JP14, JP15: (no value), trainlib:CON10M
- JP1, JP2, JP3, JP5, JP6: value (none) -> M08-SCREW; device SPCoast:1X08_LOCK -> trainlib:1X08_TERMINAL
- JP7: device jumper:JP2W -> jumper:JP3Q
- moved JP10 400.8 mm to (69.8, 71.1)
- moved JP9 381.2 mm to (59.7, 71.1)
- moved JP8 357.8 mm to (26.7, 71.1)
- moved SJ8 303.2 mm to (81.3, 15.2), flipped to the bottom
- moved SJ7 301.2 mm to (81.3, 11.4), flipped to the bottom
- moved SJ10 299.8 mm to (81.3, 7.62), flipped to the bottom
- moved SJ11 298.6 mm to (81.3, 3.81), flipped to the bottom
- moved SJ9 278.2 mm to (15.2, 24.1), flipped to the bottom
- moved SJ12 278.1 mm to (10.2, 24.1), flipped to the bottom
- moved SJ3 223.8 mm to (68.6, 20.3), flipped to the bottom
- moved SJ2 211.2 mm to (11.4, 17.8), flipped to the bottom
- moved SJ4 211.2 mm to (11.4, 2.54), flipped to the bottom
- moved SJ5 211.2 mm to (11.4, 7.62), flipped to the bottom
- moved SJ6 211.2 mm to (11.4, 12.7), flipped to the bottom
- moved SJ1 204.2 mm to (7.62, 17.8), flipped to the bottom
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Connections:
- removed net N$43: AP1509.2, D1.C, L1.2
- new net SW: AP1509.2, D1.C, IC10.7, L1.2
- net +12V: now also IC10.5
- net +5V: now also IC10.1
- net GND: now also IC10.2, IC10.3, IC10.4
- net N$14: now also JP3.7, RN4.7; no longer JP3.2, RN4.2
- net N$15: now also JP3.6, RN4.6; no longer JP3.3, RN4.3
- net N$16: now also JP3.5, RN4.5; no longer JP3.4, RN4.4
- net N$19: now also JP3.4, RN4.4; no longer JP3.5, RN4.5
- net N$20: now also JP3.3, RN4.3; no longer JP3.6, RN4.6
- net N$21: now also JP3.2, RN4.2; no longer JP3.7, RN4.7
- net N$22: now also JP3.1, RN4.1; no longer JP3.8, RN4.8
- net N$23: now also RN4.9; no longer RN4.16
- net N$24: now also RN4.10; no longer RN4.15
- net N$25: now also JP2.8, RN1.8; no longer JP2.1, RN1.1
- net N$26: now also JP2.7, RN1.7; no longer JP2.2, RN1.2
- net N$27: now also JP2.6, RN1.6; no longer JP2.3, RN1.3
- net N$28: now also JP2.5, RN1.5; no longer JP2.4, RN1.4
- net N$29: now also RN4.11; no longer RN4.14
- net N$30: now also RN4.12; no longer RN4.13
- net N$31: now also RN4.13; no longer RN4.12
- net N$32: now also RN4.14; no longer RN4.11
- net N$33: now also JP2.4, RN1.4; no longer JP2.5, RN1.5
- net N$34: now also JP2.3, RN1.3; no longer JP2.6, RN1.6
- net N$35: now also JP2.2, RN1.2; no longer JP2.7, RN1.7
- net N$36: now also JP2.1, RN1.1; no longer JP2.8, RN1.8
- net N$37: now also RN4.15; no longer RN4.10
- net N$38: now also RN4.16; no longer RN4.9
- net N$44: now also RN1.9; no longer RN1.16
- net N$47: now also RN1.10; no longer RN1.15
- net N$48: now also RN1.11; no longer RN1.14
- net N$49: now also RN1.12; no longer RN1.13
- net N$50: now also RN1.13; no longer RN1.12
- net N$51: now also RN1.14; no longer RN1.11
- net N$52: now also RN1.15; no longer RN1.10
- net N$53: now also RN1.16; no longer RN1.9
- net N$6: now also JP3.8, RN4.8; no longer JP3.1, RN4.1
