File: eagle/nucleo-io-board/io-board-a-4.sch (EAGLE design)
At the start: 52 parts, among them IC1 74166N, IC3 74HCT595N, IC4 74166N, IC5 74HCT595N, IC6 LM324N, IC7 PCA82C250, IC9 LM324N, J1 RJ45-JACKRJ45-PULSE-E5J00, J2 RJ45-JACKRJ45-PULSE-E5J00, J3 DCJ0202

Commit message: More work on the nucleo io board.
Parts:
- added IC10: LM2574N-5.0, linear:LM2574N-5.0
- added JP11: (no value), jumper:JP3Q
- added JP12: (no value), pinhead:PINHD-2X5
- added JP13, JP14, JP15: (no value), trainlib:PINHD-2X5CN
- JP1, JP2, JP3, JP5, JP6: value (none) -> M08-SCREW; device SPCoast:M08LOCK -> trainlib:M08-SCREW
- JP7: device jumper:JP2W -> jumper:JP3Q
Connections:
- removed net N$43: AP1509.VOUT, D1.C, L1.2
- new net SW: AP1509.VOUT, D1.C, IC10.OUT, L1.2
- net +12V: now also IC10.IN
- net +5V: now also IC10.FB
- net GND: now also IC10.!ON/OFF, IC10.GND@PWR, IC10.GNDSIG
- net N$14: now also JP3.7, RN4G.1; no longer JP3.2, RN4B.1
- net N$15: now also JP3.6, RN4F.1; no longer JP3.3, RN4C.1
- net N$16: now also JP3.5, RN4E.1; no longer JP3.4, RN4D.1
- net N$19: now also JP3.4, RN4D.1; no longer JP3.5, RN4E.1
- net N$20: now also JP3.3, RN4C.1; no longer JP3.6, RN4F.1
- net N$21: now also JP3.2, RN4B.1; no longer JP3.7, RN4G.1
- net N$22: now also JP3.1, RN4A.1; no longer JP3.8, RN4H.1
- net N$23: now also RN4H.2; no longer RN4A.2
- net N$24: now also RN4G.2; no longer RN4B.2
- net N$25: now also JP2.8, RN1H.1; no longer JP2.1, RN1A.1
- net N$26: now also JP2.7, RN1G.1; no longer JP2.2, RN1B.1
- net N$27: now also JP2.6, RN1F.1; no longer JP2.3, RN1C.1
- net N$28: now also JP2.5, RN1E.1; no longer JP2.4, RN1D.1
- net N$29: now also RN4F.2; no longer RN4C.2
- net N$30: now also RN4E.2; no longer RN4D.2
- net N$31: now also RN4D.2; no longer RN4E.2
- net N$32: now also RN4C.2; no longer RN4F.2
- net N$33: now also JP2.4, RN1D.1; no longer JP2.5, RN1E.1
- net N$34: now also JP2.3, RN1C.1; no longer JP2.6, RN1F.1
- net N$35: now also JP2.2, RN1B.1; no longer JP2.7, RN1G.1
- net N$36: now also JP2.1, RN1A.1; no longer JP2.8, RN1H.1
- net N$37: now also RN4B.2; no longer RN4G.2
- net N$38: now also RN4A.2; no longer RN4H.2
- net N$44: now also RN1H.2; no longer RN1A.2
- net N$47: now also RN1G.2; no longer RN1B.2
- net N$48: now also RN1F.2; no longer RN1C.2
- net N$49: now also RN1E.2; no longer RN1D.2
- net N$50: now also RN1D.2; no longer RN1E.2
- net N$51: now also RN1C.2; no longer RN1F.2
- net N$52: now also RN1B.2; no longer RN1G.2
- net N$53: now also RN1A.2; no longer RN1H.2
- net N$6: now also JP3.8, RN4H.1; no longer JP3.1, RN4A.1
Other:
- moved on the sheet: AP1509, C1, C2, D1, JP2, JP3, L1, RN1, RN4
