File: eagle/nucleo-io-board/io-board-a-5.brd (EAGLE design)
At the start: 100 x 80 mm, 52 parts, among them IC1 74166N, IC3 74HCT595N, IC4 74166N, IC5 74HCT595N, IC6 LM324N, IC7 PCA82C250, IC9 LM324N, J1 RJ45-JACKRJ45-PULSE-E5J00, J2 RJ45-JACKRJ45-PULSE-E5J00, J3 DCJ0202

Commit message: More work on the nucleo io board.
Parts:
- added IC10: LM2574N-5.0, linear:DIL08
- added JP11: (no value), jumper:JP3Q
- added JP13, JP14, JP15: (no value), trainlib:CON10M
- JP1, JP2, JP3, JP5, JP6: value (none) -> M08-SCREW; device SPCoast:1X08_LOCK -> trainlib:1X08_TERMINAL
- JP7: device jumper:JP2W -> jumper:JP3Q
- moved JP10 400.8 mm to (69.8, 71.1)
- moved JP9 381.2 mm to (59.7, 71.1)
- moved JP8 357.8 mm to (26.7, 71.1)
- moved SJ8 303.2 mm to (81.3, 15.2), flipped to the bottom
- moved SJ7 301.2 mm to (81.3, 11.4), flipped to the bottom
- moved SJ10 299.8 mm to (81.3, 7.62), flipped to the bottom
- moved SJ11 298.6 mm to (81.3, 3.81), flipped to the bottom
- moved SJ12 268.3 mm to (52.1, 11.4), flipped to the bottom, turned to 270 degrees
- moved SJ9 267.2 mm to (38.1, 11.4), flipped to the bottom, turned to 270 degrees
- moved SJ4 233.0 mm to (57.1, 11.4), flipped to the bottom, turned to 270 degrees
- moved SJ5 229.8 mm to (61.0, 11.4), flipped to the bottom, turned to 270 degrees
- moved SJ6 226.7 mm to (64.8, 11.4), flipped to the bottom, turned to 270 degrees
- moved SJ2 225.5 mm to (72.4, 11.4), flipped to the bottom, turned to 270 degrees
- moved SJ3 219.4 mm to (76.2, 11.4), flipped to the bottom, turned to 270 degrees
- moved SJ1 216.4 mm to (69.8, 11.4), flipped to the bottom, turned to 270 degrees
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Connections:
- removed net N$16: JP3.4, RN4.4, RN5.5
- removed net N$27: JP2.3, RN1.3, RN2.4
- removed net N$43: AP1509.2, D1.C, L1.2
- removed net N$65: IC6.8, JP5.7
- new net N$83: JP13.7, JP3.5, RN4.5, RN5.5
- new net N$84: JP13.2, JP3.2, RN4.2, RN5.8
- new net N$90: IC6.8, JP15.9, JP5.7
- new net SW: AP1509.2, D1.C, IC10.7, L1.2
- net +12V: now also IC10.5
- net +5V: now also IC10.1
- net GND: now also IC10.2, IC10.3, IC10.4
- net N$14: now also JP13.9, JP3.7, RN4.7; no longer JP3.2, RN4.2
- net N$15: now also JP13.8, JP3.6, RN4.6; no longer JP3.3, RN4.3
- net N$19: now also JP13.4, JP3.4, RN4.4; no longer JP3.5, RN4.5
- net N$20: now also JP13.3, JP3.3, RN4.3; no longer JP3.6, RN4.6
- net N$21: now also JP14.8, JP2.6, RN1.6, RN2.4; no longer JP3.7, RN4.7, RN5.8
- net N$22: now also JP13.1, JP3.1, RN4.1; no longer JP3.8, RN4.8
- net N$23: now also RN4.9; no longer RN4.16
- net N$24: now also RN4.10; no longer RN4.15
- net N$25: now also JP14.10, JP2.8, RN1.8; no longer JP2.1, RN1.1
- net N$26: now also JP14.9, JP2.7, RN1.7; no longer JP2.2, RN1.2
- net N$28: now also JP14.7, JP2.5, RN1.5; no longer JP2.4, RN1.4
- net N$29: now also RN4.11; no longer RN4.14
- net N$30: now also RN4.12; no longer RN4.13
- net N$31: now also RN4.13; no longer RN4.12
- net N$32: now also RN4.14; no longer RN4.11
- net N$33: now also JP14.4, JP2.4, RN1.4; no longer JP2.5, RN1.5
- net N$34: now also JP14.3, JP2.3, RN1.3; no longer JP2.6, RN1.6
- net N$35: now also JP14.2, JP2.2, RN1.2; no longer JP2.7, RN1.7
- net N$36: now also JP14.1, JP2.1, RN1.1; no longer JP2.8, RN1.8
- net N$37: now also RN4.15; no longer RN4.10
- net N$38: now also RN4.16; no longer RN4.9
- net N$44: now also RN1.9; no longer RN1.16
- net N$46: now also JP15.2
- net N$47: now also RN1.10; no longer RN1.15
- net N$48: now also RN1.11; no longer RN1.14
- net N$49: now also RN1.12; no longer RN1.13
- net N$50: now also RN1.13; no longer RN1.12
- net N$51: now also RN1.14; no longer RN1.11
- net N$52: now also RN1.15; no longer RN1.10
- net N$53: now also RN1.16; no longer RN1.9
- net N$6: now also JP13.10, JP3.8, RN4.8; no longer JP3.1, RN4.1
- net N$60: now also JP15.8
- net N$63: now also JP15.10
- net N$64: now also JP15.7
- net N$80: now also JP15.4
- net N$81: now also JP15.1
- net N$82: now also JP15.3
