File: eagle/nucleo-io-board/io-board-a-6.sch (EAGLE design)
At the start: 52 parts, among them IC1 74166N, IC3 74HCT595N, IC4 74166N, IC5 74HCT595N, IC6 LM324N, IC7 PCA82C250, IC9 LM324N, J1 RJ45-JACKRJ45-PULSE-E5J00, J2 RJ45-JACKRJ45-PULSE-E5J00, J3 DCJ0202

Commit message: More work on the nucleo io board.
Parts:
- added IC10: LM2574N-5.0, linear:LM2574N-5.0
- added JP11: (no value), jumper:JP3Q
- added JP13, JP14, JP15: (no value), trainlib:PINHD-2X5CN
- added Q1, Q2, Q3, Q4, Q5, Q6, Q7, Q8: BSS123, transistor-small-signal:BSS123
- added R10, R3, R4, R5, R6, R7, R8, R9: (no value), rcl:R-US_R0603
- IC2, IC8: device uln-udn:ULN2803A -> trainlib:ULN2803A
- JP1, JP2, JP3, JP5, JP6: value (none) -> M08-SCREW; device SPCoast:M08LOCK -> trainlib:M08-SCREW
- JP7: device jumper:JP2W -> jumper:JP3Q
Connections:
- new net N$78: Q1.G, R3.2
- new net N$79: Q2.G, R4.2
- new net N$83: JP13.7, JP3.5, RN4E.1, RN5.5
- new net N$84: JP13.2, JP3.2, RN4B.1, RN5.8
- new net N$85: Q8.G, R10.2
- new net N$88: Q3.G, R5.2
- new net N$90: IC6C.OUT, JP15.9, JP5.7
- new net SW: AP1509.VOUT, D1.C, IC10.OUT, L1.2
- net +12V: now also IC10.IN
- net +5V: now also IC10.FB
- net GND: now also IC10.!ON/OFF, IC10.GND@PWR, IC10.GNDSIG, Q1.S, Q2.S, Q3.S, Q4.S, Q5.S, Q6.S, Q7.S, Q8.S
- net N$1: now also R3.1
- net N$10: now also R6.1
- net N$11: now also Q4.D
- net N$12: now also R7.1
- net N$13: now also Q5.D
- net N$14: now also JP13.9, JP3.7, RN4G.1; no longer JP3.2, RN4B.1
- net N$15: now also JP13.8, JP3.6, RN4F.1; no longer JP3.3, RN4C.1
- net N$16: now also Q4.G, R6.2; no longer JP3.4, RN4D.1, RN5.5
- net N$17: now also R8.1
- net N$18: now also Q6.D
- net N$19: now also JP13.4, JP3.4, RN4D.1; no longer JP3.5, RN4E.1
- net N$2: now also Q1.D
- net N$20: now also JP13.3, JP3.3, RN4C.1; no longer JP3.6, RN4F.1
- net N$21: now also JP14.8, JP2.6, RN1F.1, RN2.4; no longer JP3.7, RN4G.1, RN5.8
- net N$22: now also JP13.1, JP3.1, RN4A.1; no longer JP3.8, RN4H.1
- net N$23: now also RN4H.2; no longer RN4A.2
- net N$24: now also RN4G.2; no longer RN4B.2
- net N$25: now also JP14.10, JP2.8, RN1H.1; no longer JP2.1, RN1A.1
- net N$26: now also JP14.9, JP2.7, RN1G.1; no longer JP2.2, RN1B.1
- net N$27: now also Q5.G, R7.2; no longer JP2.3, RN1C.1, RN2.4
- net N$28: now also JP14.7, JP2.5, RN1E.1; no longer JP2.4, RN1D.1
- net N$29: now also RN4F.2; no longer RN4C.2
- net N$3: now also R4.1
- net N$30: now also RN4E.2; no longer RN4D.2
- net N$31: now also RN4D.2; no longer RN4E.2
- net N$32: now also RN4C.2; no longer RN4F.2
- net N$33: now also JP14.4, JP2.4, RN1D.1; no longer JP2.5, RN1E.1
- net N$34: now also JP14.3, JP2.3, RN1C.1; no longer JP2.6, RN1F.1
- net N$35: now also JP14.2, JP2.2, RN1B.1; no longer JP2.7, RN1G.1
- net N$36: now also JP14.1, JP2.1, RN1A.1; no longer JP2.8, RN1H.1
- net N$37: now also RN4B.2; no longer RN4G.2
- net N$38: now also RN4A.2; no longer RN4H.2
- net N$39: now also R9.1
- net N$40: now also Q7.D
- net N$41: now also R10.1
- net N$42: now also Q8.D
- net N$43: now also Q6.G, R8.2; no longer AP1509.VOUT, D1.C, L1.2
- net N$44: now also RN1H.2; no longer RN1A.2
- net N$46: now also JP15.2
- net N$47: now also RN1G.2; no longer RN1B.2
- net N$48: now also RN1F.2; no longer RN1C.2
- net N$49: now also RN1E.2; no longer RN1D.2
- net N$50: now also RN1D.2; no longer RN1E.2
- net N$51: now also RN1C.2; no longer RN1F.2
- net N$52: now also RN1B.2; no longer RN1G.2
- net N$53: now also RN1A.2; no longer RN1H.2
- net N$6: now also JP13.10, JP3.8, RN4H.1; no longer JP3.1, RN4A.1
- net N$60: now also JP15.8
- net N$63: now also JP15.10
- net N$64: now also JP15.7
- net N$65: now also Q7.G, R9.2; no longer IC6C.OUT, JP5.7
- net N$7: now also Q2.D
- net N$8: now also R5.1
- net N$80: now also JP15.4
- net N$81: now also JP15.1
- net N$82: now also JP15.3
- net N$9: now also Q3.D
Other:
- moved on the sheet: AP1509, C1, C2, D1, JP2, JP3, JP5, L1, RN1, RN4
