File: eagle/nucleo-io-board/io-board-a-8.sch (EAGLE design)
At the start: 52 parts, among them IC1 74166N, IC3 74HCT595N, IC4 74166N, IC5 74HCT595N, IC6 LM324N, IC7 PCA82C250, IC9 LM324N, J1 RJ45-JACKRJ45-PULSE-E5J00, J2 RJ45-JACKRJ45-PULSE-E5J00, J3 DCJ0202

Commit message: More work on the nucleo io board.
Parts:
- added IC10: LM2574N-5.0, linear:LM2574N-5.0
- added JP11: (no value), jumper:JP3Q
- added JP13, JP14, JP15: (no value), trainlib:PINHD-2X5CN
- added Q1, Q10, Q11, Q12, Q13, Q14, Q15, Q16, Q2, Q3, Q4, Q5, Q6, Q7, Q8, Q9: BSS123, transistor-small-signal:BSS123
- added R10, R11, R12, R13, R14, R15, R16, R17, R18, R3, R4, R5, R6, R7, R8, R9: (no value), rcl:R-US_R0603
- added R19, R20: (no value), rcl:R-US_R0805
- added U$2, U$3, U$4, U$5: TC4426APDIP, trainlib:TC4426APDIP
- IC2, IC8: device uln-udn:ULN2803A -> trainlib:ULN2803A
- JP1, JP2, JP3, JP5, JP6: value (none) -> M08-SCREW; device SPCoast:M08LOCK -> trainlib:M08-SCREW
- JP7: device jumper:JP2W -> jumper:JP3Q
- SJ3, SJ9: value SJ-C -> (none)
Connections:
- net !OSS renamed OLAT
- net N$45 renamed CMPREF
- removed net N$46: IC9B.OUT, JP5.2
- removed net N$57: IC8.O1, JP6.1
- removed net N$58: IC3A.QB, IC8.I2
- removed net N$59: IC8.O2, JP6.2
- removed net N$60: IC6B.OUT, JP5.6
- removed net N$61: IC3A.QC, IC8.I3
- removed net N$62: IC8.O3, JP6.3
- removed net N$63: IC6D.OUT, JP5.8
- removed net N$64: IC6A.OUT, JP5.5
- removed net N$66: IC3A.QD, IC8.I4
- removed net N$67: IC8.O4, JP6.4
- removed net N$68: IC3A.QE, IC8.I5
- removed net N$69: IC8.O5, JP6.5
- removed net N$70: IC3A.QF, IC8.I6
- removed net N$71: IC8.O6, JP6.6
- removed net N$72: IC3A.QG, IC8.I7
- removed net N$73: IC8.O7, JP6.7
- removed net N$74: IC3A.QH, IC8.I8
- removed net N$80: IC9D.OUT, JP5.4
- removed net N$81: IC9A.OUT, JP5.1
- removed net N$82: IC9C.OUT, JP5.3
- new net N$100: IC3A.QG, IC8.I7, R17.1
- new net N$101: IC8.O7, JP6.7, Q15.D
- new net N$102: IC3A.QH, IC8.I8, R18.1
- new net N$104: Q9.G, R11.2
- new net N$105: Q10.G, R12.2
- new net N$106: Q11.G, R13.2
- new net N$107: Q12.G, R14.2
- new net N$108: Q13.G, R15.2
- new net N$109: Q14.G, R16.2
- new net N$110: Q15.G, R17.2
- new net N$111: Q16.G, R18.2
- new net N$78: Q1.G, R3.2
- new net N$79: Q2.G, R4.2
- new net N$83: JP13.7, JP3.5, RN4E.1, RN5.5
- new net N$84: JP13.2, JP3.2, RN4B.1, RN5.8
- new net N$85: Q8.G, R10.2
- new net N$87: IC8.O1, JP6.1, Q9.D
- new net N$88: Q3.G, R5.2
- new net N$89: IC3A.QB, IC8.I2, R12.1
- new net N$91: IC8.O2, JP6.2, Q10.D
- new net N$92: IC3A.QC, IC8.I3, R13.1
- new net N$93: IC8.O3, JP6.3, Q11.D
- new net N$94: IC3A.QD, IC8.I4, R14.1
- new net N$95: IC8.O4, JP6.4, Q12.D
- new net N$96: IC3A.QE, IC8.I5, R15.1
- new net N$97: IC8.O5, JP6.5, Q13.D
- new net N$98: IC3A.QF, IC8.I6, R16.1
- new net N$99: IC8.O6, JP6.6, Q14.D
- new net SLNK1: IC3A.SER, IC5A.QH*
- new net SW: AP1509.VOUT, D1.C, IC10.OUT, L1.2
- new net TIN1: IC9A.+IN, U$2G$2.I
- new net TIN2: IC9B.+IN, U$2G$3.I
- new net TIN3: IC9C.+IN, U$3G$2.I
- new net TIN4: IC9D.+IN, U$3G$3.I
- new net TIN5: IC6A.+IN, U$4G$2.I
- new net TIN6: IC6B.+IN, U$4G$3.I
- new net TIN7: IC6C.+IN, U$5G$2.I
- new net TIN8: IC6D.+IN, U$5G$3.I
- new net TOUT1: IC9A.OUT, JP15.1, JP5.1, U$2G$2.O
- new net TOUT2: IC9B.OUT, JP15.2, JP5.2, U$2G$3.O
- new net TOUT3: IC9C.OUT, JP15.3, JP5.3, U$3G$2.O
- new net TOUT4: IC9D.OUT, JP15.4, JP5.4, U$3G$3.O
- new net TOUT5: IC6A.OUT, JP15.7, JP5.5, U$4G$2.O
- new net TOUT6: IC6B.OUT, JP15.8, JP5.6, U$4G$3.O
- new net TOUT7: IC6C.OUT, JP15.9, JP5.7, U$5G$2.O
- new net TOUT8: IC6D.OUT, JP15.10, JP5.8, U$5G$3.O
- net +12V: now also IC10.IN, U$2G$1.VDD, U$3G$1.VDD, U$4G$1.VDD, U$5G$1.VDD
- net +5V: now also IC10.FB, R19.2, R20.2
- net GND: now also IC10.!ON/OFF, IC10.GND@PWR, IC10.GNDSIG, Q1.S, Q10.S, Q11.S, Q12.S, Q13.S, Q14.S, Q15.S, Q16.S, Q2.S, Q3.S, Q4.S, Q5.S, Q6.S, Q7.S, Q8.S, Q9.S, U$2G$1.VSS, U$3G$1.VSS, U$4G$1.VSS, U$5G$1.VSS
- net MISO: now also U$1.PB4
- net MOSI: now also R20.1, U$1.PB5; no longer IC3A.SER
- net N$1: now also R3.1
- net N$10: now also R6.1
- net N$11: now also Q4.D
- net N$12: now also R7.1
- net N$13: now also Q5.D
- net N$14: now also JP13.9, JP3.7, RN4G.1; no longer JP3.2, RN4B.1
- net N$15: now also JP13.8, JP3.6, RN4F.1; no longer JP3.3, RN4C.1
- net N$16: now also Q4.G, R6.2; no longer JP3.4, RN4D.1, RN5.5
- net N$17: now also R8.1
- net N$18: now also Q6.D
- net N$19: now also JP13.4, JP3.4, RN4D.1; no longer JP3.5, RN4E.1
- net N$2: now also Q1.D
- net N$20: now also JP13.3, JP3.3, RN4C.1; no longer JP3.6, RN4F.1
- net N$21: now also JP14.8, JP2.6, RN1F.1, RN2.4; no longer JP3.7, RN4G.1, RN5.8
- net N$22: now also JP13.1, JP3.1, RN4A.1; no longer JP3.8, RN4H.1
- net N$23: now also RN4H.2; no longer RN4A.2
- net N$24: now also RN4G.2; no longer RN4B.2
- net N$25: now also JP14.10, JP2.8, RN1H.1; no longer JP2.1, RN1A.1
- net N$26: now also JP14.9, JP2.7, RN1G.1; no longer JP2.2, RN1B.1
- net N$27: now also Q5.G, R7.2; no longer JP2.3, RN1C.1, RN2.4
- net N$28: now also JP14.7, JP2.5, RN1E.1; no longer JP2.4, RN1D.1
- net N$29: now also RN4F.2; no longer RN4C.2
- net N$3: now also R4.1
- net N$30: now also RN4E.2; no longer RN4D.2
- net N$31: now also RN4D.2; no longer RN4E.2
- net N$32: now also RN4C.2; no longer RN4F.2
- net N$33: now also JP14.4, JP2.4, RN1D.1; no longer JP2.5, RN1E.1
- net N$34: now also JP14.3, JP2.3, RN1C.1; no longer JP2.6, RN1F.1
- net N$35: now also JP14.2, JP2.2, RN1B.1; no longer JP2.7, RN1G.1
- net N$36: now also JP14.1, JP2.1, RN1A.1; no longer JP2.8, RN1H.1
- net N$37: now also RN4B.2; no longer RN4G.2
- net N$38: now also RN4A.2; no longer RN4H.2
- net N$39: now also R9.1
- net N$40: now also Q7.D
- net N$41: now also R10.1
- net N$42: now also Q8.D
- net N$43: now also Q6.G, R8.2; no longer AP1509.VOUT, D1.C, L1.2
- net N$44: now also RN1H.2; no longer RN1A.2
- net N$47: now also RN1G.2; no longer RN1B.2
- net N$48: now also RN1F.2; no longer RN1C.2
- net N$49: now also RN1E.2; no longer RN1D.2
- net N$50: now also RN1D.2; no longer RN1E.2
- net N$51: now also RN1C.2; no longer RN1F.2
- net N$52: now also RN1B.2; no longer RN1G.2
- net N$53: now also RN1A.2; no longer RN1H.2
- net N$56: now also R11.1
- net N$6: now also JP13.10, JP3.8, RN4H.1; no longer JP3.1, RN4A.1
- net N$65: now also Q7.G, R9.2; no longer IC6C.OUT, JP5.7
- net N$7: now also Q2.D
- net N$75: now also Q16.D
- net N$8: now also R5.1
- net N$9: now also Q3.D
- net SCK: now also R19.1, U$1.PB3
Other:
- moved on the sheet: AP1509, C1, C2, D1, IC2, IC5, IC5P, JP1, JP2, JP3, JP5, L1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
