File: eagle/nucleo-io-board/io-board-d-7.brd (EAGLE design)
At the start: 100 x 80 mm, 163 parts, among them J1 RJ45-JACK, J2 RJ45-JACK, J3 DCJ0202, U1 74HC166, U10 LM324N, U11 74AHCT595N, U13 74AHCT595N, U2 74HC166, U3 TC4426/28, U4 TC4426/28, U5 TC4426/28, U6 TC4426/28, U7 CAN-TXR-PDIP, U7B CAN-TXR-SO8, U8 AP1509-50, U8B LM2574N-5.0, U9 LM324N, X1 M08-SCREW, X2 M08-SCREW, X3 M08-SCREW, X4 PORTD, X5 PORTE

Commit message: Rev A final version.
Routing:
- net V+: track 111.9 -> 109.0 mm
- net CANL: track 117.5 -> 118.4 mm
- net +5V: track 429.5 -> 430.4 mm
- net CANH: track 121.8 -> 122.4 mm
- net GND: track 773.8 -> 774.1 mm, vias 196 -> 203
