File: eagle/nucleo-io-board/io-board-f-5.sch (EAGLE design)
At the start: 166 parts, among them IC1 LM2574N-5.0, IC2 CAN-TXR-SO8, J1 DCJ0202, P1 9-15V DC, Q1 BSS123, Q10 BSS123, Q11 BSS123, Q12 BSS123, Q13 BSS123, Q14 BSS123, Q15 BSS123, Q16 BSS123, Q2 BSS123, Q3 BSS123, Q4 BSS123, Q5 BSS123, Q6 BSS123, Q7 BSS123, Q8 BSS123, Q9 BSS123, U1 CAN-TXR-PDIP, U10 TC4426/28, U11 74AHCT595N, U13 74AHCT595N, U2 AP1509-50, U3 74HC166, U4 74HC166, U5 TC4426/28, U6 LM324N, U7 TC4426/28, U8 TC4426/28, U9 LM324N, X1 RJ45-JACK, X2 RJ45-JACK, X3 M08-SCREW, X4 M08-SCREW, X6 M08-SCREW, X7 PORTD, X8 PORTE

Commit message: New revisions to fix comments from the review process.
Parts:
- added D5: (no value), diode:DIODE-DO41-7.6
- added D6: DIODEDO-214AA-NODOC, trainlib:DIODEDO-214AA-NODOC
- added X9: (no value), SPCoast:CONNECTOR-M023.5MM-LOCK
- U10, U5, U7, U8: value TC4426/28 -> TC4427
Connections:
- new net N$4: D5.A, D6.A, J1.1, X9.1
- net +12V: now also D5.C, D6.C; no longer J1.1
- net GND: now also X9.2
Changed lines of the file:
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@@
 <part name="P+4" library="supply1" library_urn="urn:adsk.eagle:library:371" deviceset="+5V" device=""/>
 <part name="R4" library="rcl" library_urn="urn:adsk.eagle:library:334" deviceset="R-US_" device="R0805" package3d_urn="urn:adsk.eagle:package:23553/2"/>
-<part name="U8" library="trainlib" deviceset="TC4426A" device="PDIP" value="TC4426/28"/>
-<part name="U10" library="trainlib" deviceset="TC4426A" device="PDIP" value="TC4426/28"/>
-<part name="U5" library="trainlib" deviceset="TC4426A" device="PDIP" value="TC4426/28"/>
-<part name="U7" library="trainlib" deviceset="TC4426A" device="PDIP" value="TC4426/28"/>
+<part name="U8" library="trainlib" deviceset="TC4426A" device="PDIP" value="TC4427"/>
+<part name="U10" library="trainlib" deviceset="TC4426A" device="PDIP" value="TC4427"/>
+<part name="U5" library="trainlib" deviceset="TC4426A" device="PDIP" value="TC4427"/>
+<part name="U7" library="trainlib" deviceset="TC4426A" device="PDIP" value="TC4427"/>
 <part name="SUPPLY34" library="supply2" library_urn="urn:adsk.eagle:library:372" deviceset="GND" device=""/>
 <part name="P+24" library="supply1" library_urn="urn:adsk.eagle:library:371" deviceset="+12V" device=""/>
@@
 <part name="LOGO1" library="SPCoast" deviceset="DOC-OSHW-LOGO" device="M" value="DOC-OSHW-LOGOM"/>
 <part name="SJ20" library="trainlib" deviceset="SJ" device="RND2"/>
+<part name="D5" library="diode" library_urn="urn:adsk.eagle:library:210" deviceset="DIODE-" device="DO41-7.6" package3d_urn="urn:adsk.eagle:package:43421/1"/>
+<part name="D6" library="trainlib" deviceset="DIODE" device="DO-214AA-NODOC"/>
+<part name="X9" library="SPCoast" deviceset="CONNECTOR-M02" device="3.5MM-LOCK"/>
 </parts>
 <sheets>
@@
 <instance part="H3" gate="G$1" x="195.58" y="-157.48"/>
 <instance part="H4" gate="G$1" x="208.28" y="-157.48"/>
-<instance part="P+17" gate="1" x="33.02" y="-104.14"/>
+<instance part="P+17" gate="1" x="20.32" y="-88.9"/>
 <instance part="J1" gate="G$1" x="15.24" y="-111.76"/>
-<instance part="SUPPLY20" gate="GND" x="25.4" y="-119.38"/>
+<instance part="SUPPLY20" gate="GND" x="25.4" y="-129.54"/>
 <instance part="X2" gate="G$1" x="22.86" y="-58.42" rot="MR0"/>
 <instance part="X1" gate="G$1" x="22.86" y="-35.56" rot="MR0"/>
@@
 <instance part="LOGO1" gate="LOGO" x="213.36" y="-111.76"/>
 <instance part="SJ20" gate="1" x="218.44" y="132.08" rot="R180"/>
+<instance part="D5" gate="G$1" x="35.56" y="-111.76" smashed="yes">
+<attribute name="NAME" x="38.1" y="-111.2774" size="1.778" layer="95"/>
+<attribute name="VALUE" x="38.1" y="-114.0714" size="1.778" layer="96"/>
+</instance>
+<instance part="D6" gate="D$1" x="35.56" y="-106.68" smashed="yes">
+<attribute name="NAME" x="38.1" y="-106.1974" size="1.778" layer="95"/>
+</instance>
+<instance part="X9" gate="G$1" x="40.64" y="-121.92" rot="R180"/>
 </instances>
 <busses>
@@
 <segment>
 <pinref part="JP7" gate="B1" pin="2"/>
-<wire x1="27.94" y1="-93.98" x2="25.4" y2="-93.98" width="0.1524" layer="91"/>
 <pinref part="P+17" gate="1" pin="+12V"/>
-<wire x1="33.02" y1="-106.68" x2="33.02" y2="-109.22" width="0.1524" layer="91"/>
-<pinref part="J1" gate="G$1" pin="1"/>
-<wire x1="33.02" y1="-109.22" x2="25.4" y2="-109.22" width="0.1524" layer="91"/>
-<wire x1="25.4" y1="-109.22" x2="22.86" y2="-109.22" width="0.1524" layer="91"/>
-<wire x1="25.4" y1="-93.98" x2="25.4" y2="-109.22" width="0.1524" layer="91"/>
-<junction x="25.4" y="-109.22"/>
+<wire x1="20.32" y1="-91.44" x2="20.32" y2="-93.98" width="0.1524" layer="91"/>
+<wire x1="20.32" y1="-93.98" x2="27.94" y2="-93.98" width="0.1524" layer="91"/>
+<pinref part="D5" gate="G$1" pin="C"/>
+<wire x1="38.1" y1="-111.76" x2="43.18" y2="-111.76" width="0.1524" layer="91"/>
+<wire x1="43.18" y1="-111.76" x2="43.18" y2="-106.68" width="0.1524" layer="91"/>
+<wire x1="43.18" y1="-106.68" x2="43.18" y2="-101.6" width="0.1524" layer="91"/>
+<wire x1="43.18" y1="-101.6" x2="20.32" y2="-101.6" width="0.1524" layer="91"/>
+<wire x1="20.32" y1="-101.6" x2="20.32" y2="-93.98" width="0.1524" layer="91"/>
+<junction x="20.32" y="-93.98"/>
+<pinref part="D6" gate="D$1" pin="C"/>
+<wire x1="38.1" y1="-106.68" x2="43.18" y2="-106.68" width="0.1524" layer="91"/>
+<junction x="43.18" y="-106.68"/>
 </segment>
 <segment>
@@
 <segment>
 <pinref part="SUPPLY20" gate="GND" pin="GND"/>
-<wire x1="25.4" y1="-114.3" x2="25.4" y2="-116.84" width="0.1524" layer="91"/>
+<wire x1="25.4" y1="-114.3" x2="25.4" y2="-124.46" width="0.1524" layer="91"/>
 <pinref part="J1" gate="G$1" pin="3"/>
+<wire x1="25.4" y1="-124.46" x2="25.4" y2="-127" width="0.1524" layer="91"/>
 <wire x1="25.4" y1="-114.3" x2="22.86" y2="-114.3" width="0.1524" layer="91"/>
 <pinref part="J1" gate="G$1" pin="2"/>
@@
 <wire x1="25.4" y1="-111.76" x2="25.4" y2="-114.3" width="0.1524" layer="91"/>
 <junction x="25.4" y="-114.3"/>
+<pinref part="X9" gate="G$1" pin="2"/>
+<wire x1="35.56" y1="-124.46" x2="25.4" y2="-124.46" width="0.1524" layer="91"/>
+<junction x="25.4" y="-124.46"/>
 </segment>
 <segment>
@@
 </segment>
 </net>
+<net name="N$4" class="0">
+<segment>
+<pinref part="J1" gate="G$1" pin="1"/>
+<wire x1="22.86" y1="-109.22" x2="30.48" y2="-109.22" width="0.1524" layer="91"/>
+<pinref part="D6" gate="D$1" pin="A"/>
+<wire x1="33.02" y1="-106.68" x2="30.48" y2="-106.68" width="0.1524" layer="91"/>
+<wire x1="30.48" y1="-106.68" x2="30.48" y2="-109.22" width="0.1524" layer="91"/>
+<pinref part="D5" gate="G$1" pin="A"/>
+<wire x1="33.02" y1="-111.76" x2="30.48" y2="-111.76" width="0.1524" layer="91"/>
+<wire x1="30.48" y1="-111.76" x2="30.48" y2="-109.22" width="0.1524" layer="91"/>
+<junction x="30.48" y="-109.22"/>
+<pinref part="X9" gate="G$1" pin="1"/>
+<wire x1="35.56" y1="-121.92" x2="30.48" y2="-121.92" width="0.1524" layer="91"/>
+<wire x1="30.48" y1="-121.92" x2="30.48" y2="-111.76" width="0.1524" layer="91"/>
+<junction x="30.48" y="-111.76"/>
+</segment>
+</net>
