File: eagle/nucleo-io-board/io-board-f-9.sch (EAGLE design)
At the start: 166 parts, among them IC1 LM2574N-5.0, IC2 CAN-TXR-SO8, J1 DCJ0202, P1 9-15V DC, Q1 BSS123, Q10 BSS123, Q11 BSS123, Q12 BSS123, Q13 BSS123, Q14 BSS123, Q15 BSS123, Q16 BSS123, Q2 BSS123, Q3 BSS123, Q4 BSS123, Q5 BSS123, Q6 BSS123, Q7 BSS123, Q8 BSS123, Q9 BSS123, U1 CAN-TXR-PDIP, U10 TC4426/28, U11 74AHCT595N, U13 74AHCT595N, U2 AP1509-50, U3 74HC166, U4 74HC166, U5 TC4426/28, U6 LM324N, U7 TC4426/28, U8 TC4426/28, U9 LM324N, X1 RJ45-JACK, X2 RJ45-JACK, X3 M08-SCREW, X4 M08-SCREW, X6 M08-SCREW, X7 PORTD, X8 PORTE

Commit message: New revisions to fix comments from the review process.
Parts:
- added D5: (no value), diode:DIODE-DO41-7.6
- added D6: DIODEDO-214AA-NODOC, trainlib:DIODEDO-214AA-NODOC
- added X9: PORTE, trainlib:M09-SCREW
- D3: value (none) -> DIODEDO-214AA-NODOC; device diode:DIODE-DO41-7.6 -> trainlib:DIODEDO-214AA-NODOC
- D4: value DIODEDO-214AA-NODOC -> (none); device trainlib:DIODEDO-214AA-NODOC -> diode:DIODE-DO41-7.6
- JP10: value (none) -> PORTC
- JP8: value (none) -> PORTB
- JP9: value (none) -> PORTA
- SJ11, SJ18, SJ3: device trainlib:SJ-C -> trainlib:SJRND2
- SJ12, SJ19, SJ4: device trainlib:SJRND2 -> trainlib:SJ-C
- U10, U5, U7, U8: value TC4426/28 -> TC4427
- X3, X6: value M08-SCREW -> (none); device trainlib:M08-SCREW -> SPCoast:CONNECTOR-M023.5MM-LOCK
- X5: value (none) -> M09-SCREW; device SPCoast:CONNECTOR-M023.5MM-LOCK -> trainlib:M09-SCREW
- X7: value PORTD -> M08-SCREW; device trainlib:M09-SCREW -> trainlib:M08-SCREW
- X8: value PORTE -> PORTD
Connections:
- removed net N$36: JP8.1, R25.2, R26.2, RN1.9, RN2A.1, X3.1
- removed net N$54: G1.PB13, SJ20.2
- new net N$4: D3.A, D4.A, J1.1, X3.1
- new net N$5: JP8.10, R25.2, R26.2, RN1.9, RN2A.1, X4.1
- new net SCK2_ALT: G1.PB13, SJ2.2
- net +12V: now also D3.C, D4.C, SJ11.2, SJ18.2, SJ3.2; no longer J1.1, SJ16.2, SJ2.2, SJ9.2
- net +3V3: now also SJ6.1; no longer SJ5.1
- net +5V: now also SJ16.2, SJ9.2, X6.1; no longer SJ14.2, SJ7.2, X5.1
- net CAN_VIO: now also SJ6.2; no longer SJ5.2
- net E_MOSI: now also SJ5.2; no longer SJ3.2
- net GND: now also D5.A, D6.A, SJ13.2, SJ20.2, X3.2, X5.9, X6.2; no longer D3.A, D4.A, SJ11.2, SJ18.2, X5.2
- net LPOWA: now also SJ10.1, SJ12.1, SJ8.1; no longer SJ11.1, SJ7.1, SJ9.1
- net LPOWB: now also SJ11.1, SJ13.1, SJ9.1, X8.9; no longer SJ10.1, SJ12.1, SJ8.1, X7.9
- net MISO2: now also SJ7.2; no longer SJ6.2
- net MOSI: now also SJ14.2, SJ4.1; no longer SJ13.2, SJ3.1
- net N$101: now also X8.7; no longer X7.7
- net N$11: now also X9.4; no longer X8.4
- net N$13: now also X9.5; no longer X8.5
- net N$14: now also JP9.2, X5.7; no longer JP9.9, X4.7
- net N$15: now also JP9.3, X5.6; no longer JP9.8, X4.6
- net N$18: now also X9.6; no longer X8.6
- net N$19: now also JP9.7, X5.4; no longer JP9.4, X4.4
- net N$2: now also X9.1; no longer X8.1
- net N$20: now also JP9.8, X5.3; no longer JP9.3, X4.3
- net N$21: now also JP8.3, X4.6; no longer JP8.8, X3.6
- net N$22: now also JP9.10, X5.1; no longer JP9.1, X4.1
- net N$25: now also JP8.1, X4.8; no longer JP8.10, X3.8
- net N$26: now also JP8.2, X4.7; no longer JP8.9, X3.7
- net N$28: now also JP8.4, X4.5; no longer JP8.7, X3.5
- net N$33: now also JP8.7, X4.4; no longer JP8.4, X3.4
- net N$34: now also JP8.8, X4.3; no longer JP8.3, X3.3
- net N$35: now also JP8.9, X4.2; no longer JP8.2, X3.2
- net N$40: now also X9.7; no longer X8.7
- net N$42: now also X9.8; no longer X8.8
- net N$6: now also JP9.1, X5.8; no longer JP9.10, X4.8
- net N$60: now also SJ3.1; no longer SJ2.1
- net N$7: now also X9.2; no longer X8.2
- net N$75: now also X8.8; no longer X7.8
- net N$83: now also JP9.4, X5.5; no longer JP9.7, X4.5
- net N$84: now also JP9.9, X5.2; no longer JP9.2, X4.2
- net N$87: now also X8.1; no longer X7.1
- net N$9: now also X9.3; no longer X8.3
- net N$91: now also X8.2; no longer X7.2
- net N$93: now also X8.3; no longer X7.3
- net N$95: now also X8.4; no longer X7.4
- net N$97: now also X8.5; no longer X7.5
- net N$99: now also X8.6; no longer X7.6
- net RPOWA: now also SJ15.1, SJ17.1, SJ19.1; no longer SJ14.1, SJ16.1, SJ18.1
- net RPOWB: now also SJ16.1, SJ18.1, SJ20.1, X9.9; no longer SJ15.1, SJ17.1, SJ19.1, X8.9
- net SCK2: now also SJ2.1; no longer SJ20.1
- net SLNK1: now also SJ14.1; no longer SJ13.1
- net SLNK2: now also SJ5.1; no longer SJ4.1
- net SLNK3: now also SJ7.1; no longer SJ6.1
- net SRV5: now also G1.PC12; no longer G1.PF1-PH1
- net SRV7: now also G1.PF1-PH1; no longer G1.PC12
- net SW: now also D5.C, D6.C; no longer D3.C, D4.C
- net TOUT1: now also JP10.10, X7.1; no longer JP10.1, X6.1
- net TOUT2: now also JP10.9, X7.2; no longer JP10.2, X6.2
- net TOUT3: now also JP10.8, X7.3; no longer JP10.3, X6.3
- net TOUT4: now also JP10.7, X7.4; no longer JP10.4, X6.4
- net TOUT5: now also JP10.4, X7.5; no longer JP10.7, X6.5
- net TOUT6: now also JP10.3, X7.6; no longer JP10.8, X6.6
- net TOUT7: now also JP10.2, X7.7; no longer JP10.9, X6.7
- net TOUT8: now also JP10.1, X7.8; no longer JP10.10, X6.8
Other:
- note added: "Close both for F303RE."
- note added: "Populate only one alternative of U7 (PDIP-8) or U7B (SOIC-8) depending on the package. Example part choice: - MCP2551: R61 is 0 ohm or a slew control resistor. SJ18 open. - PCA82C250. R61 is 0 ohm or a slew control resistor. SJ18 open. - MCP2561, ATA6560/62: not recommended. - MCP2562 ATA6561/63: R61 is 0 ohm, SJ18 closed. - SN65HVD1050: R61 is 0 ohm, SJ18 open. - MCP2542FD: R61 is 0 ohm, SJ18 cl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"
- note removed: "Close for F303RE."
- note removed: "Populate only one alternative of U7 (PDIP-8) or U7B (SOIC-8) depending on the package. Example part choice: - MCP2551: R61 optional if slew rate control is needed. SJ18 open. - PCA82C250. R61 is 0 ohm or a slew control resistor. SJ18 open. - MCP2561, ATA6560/62: not recommended. - MCP2562 ATA6561/63: R61 is 0 ohm, SJ18 closed. - SN65HVD1050: R61 is 0 ohm, SJ18 open. - MCP2542FD: R61 is 0 ohm, SJ1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"
- moved on the sheet: SJ10, SJ13, SJ14, SJ15, SJ16, SJ17, SJ2, SJ20, SJ5, SJ6, SJ7, SJ8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
