File: eagle/nucleo-io-board/io-board-f-b.sch (EAGLE design)
At the start: 166 parts, among them IC1 LM2574N-5.0, IC2 CAN-TXR-SO8, J1 DCJ0202, P1 9-15V DC, Q1 BSS123, Q10 BSS123, Q11 BSS123, Q12 BSS123, Q13 BSS123, Q14 BSS123, Q15 BSS123, Q16 BSS123, Q2 BSS123, Q3 BSS123, Q4 BSS123, Q5 BSS123, Q6 BSS123, Q7 BSS123, Q8 BSS123, Q9 BSS123, U1 CAN-TXR-PDIP, U10 TC4426/28, U11 74AHCT595N, U13 74AHCT595N, U2 AP1509-50, U3 74HC166, U4 74HC166, U5 TC4426/28, U6 LM324N, U7 TC4426/28, U8 TC4426/28, U9 LM324N, X1 RJ45-JACK, X2 RJ45-JACK, X3 M08-SCREW, X4 M08-SCREW, X6 M08-SCREW, X7 PORTD, X8 PORTE

Commit message: New revisions to fix comments from the review process.
Parts:
- added D5: (no value), diode:DIODE-DO41-7.6
- added D6: DIODEDO-214AA-NODOC, trainlib:DIODEDO-214AA-NODOC
- added X9: PORTE, trainlib:M09-SCREW
- D3: value (none) -> DIODEDO-214AA-NODOC; device diode:DIODE-DO41-7.6 -> trainlib:DIODEDO-214AA-NODOC
- D4: value DIODEDO-214AA-NODOC -> (none); device trainlib:DIODEDO-214AA-NODOC -> diode:DIODE-DO41-7.6
- J1: device con-jack:DCJ0202 -> trainlib:DCJ0202
- JP10: value (none) -> PORTC
- JP8: value (none) -> PORTB
- JP9: value (none) -> PORTA
- R14, R15: value (none) -> 5k
- SJ11, SJ18, SJ3: device trainlib:SJ-C -> trainlib:SJRND2
- SJ12, SJ19, SJ4: device trainlib:SJRND2 -> trainlib:SJ-C
- U10, U5, U7, U8: value TC4426/28 -> TC4427
- X3, X6: value M08-SCREW -> (none); device trainlib:M08-SCREW -> SPCoast:CONNECTOR-M023.5MM-LOCK
- X5: value (none) -> M09-SCREW; device SPCoast:CONNECTOR-M023.5MM-LOCK -> trainlib:M09-SCREW
- X7: value PORTD -> M08-SCREW; device trainlib:M09-SCREW -> trainlib:M08-SCREW
- X8: value PORTE -> PORTD
- renumbered IC1 to U2B, IC2 to U1B
Connections:
- removed net N$36: JP8.1, R25.2, R26.2, RN1.9, RN2A.1, X3.1
- removed net N$54: G1.PB13, SJ20.2
- new net N$4: D3.A, D4.A, J1.1, J1.1B, X3.1
- new net N$5: JP8.10, R25.2, R26.2, RN1.9, RN2A.1, X4.1
- new net SCK2_ALT: G1.PB13, SJ2.2
- net +12V: now also D3.C, D4.C, SJ11.2, SJ18.2, SJ3.2; no longer J1.1, SJ16.2, SJ2.2, SJ9.2
- net +3V3: now also SJ6.1; no longer SJ5.1
- net +5V: now also SJ16.2, SJ9.2, X6.1; no longer SJ14.2, SJ7.2, X5.1
- net CAN_VIO: now also SJ6.2; no longer SJ5.2
- net E_MOSI: now also SJ5.2; no longer SJ3.2
- net GND: now also D5.A, D6.A, J1.2B, J1.3B, SJ13.2, SJ20.2, X3.2, X5.9, X6.2; no longer D3.A, D4.A, SJ11.2, SJ18.2, X5.2
- net LPOWA: now also SJ10.1, SJ12.1, SJ8.1; no longer SJ11.1, SJ7.1, SJ9.1
- net LPOWB: now also SJ11.1, SJ13.1, SJ9.1, X8.9; no longer SJ10.1, SJ12.1, SJ8.1, X7.9
- net MISO2: now also SJ7.2; no longer SJ6.2
- net MOSI: now also SJ14.2, SJ4.1; no longer SJ13.2, SJ3.1
- net N$101: now also X8.7; no longer X7.7
- net N$11: now also X9.4; no longer X8.4
- net N$13: now also X9.5; no longer X8.5
- net N$14: now also JP9.2, X5.7; no longer JP9.9, X4.7
- net N$15: now also JP9.3, X5.6; no longer JP9.8, X4.6
- net N$18: now also X9.6; no longer X8.6
- net N$19: now also JP9.7, X5.4; no longer JP9.4, X4.4
- net N$2: now also X9.1; no longer X8.1
- net N$20: now also JP9.8, X5.3; no longer JP9.3, X4.3
- net N$21: now also JP8.3, X4.6; no longer JP8.8, X3.6
- net N$22: now also JP9.10, X5.1; no longer JP9.1, X4.1
- net N$25: now also JP8.1, X4.8; no longer JP8.10, X3.8
- net N$26: now also JP8.2, X4.7; no longer JP8.9, X3.7
- net N$28: now also JP8.4, X4.5; no longer JP8.7, X3.5
- net N$33: now also JP8.7, X4.4; no longer JP8.4, X3.4
- net N$34: now also JP8.8, X4.3; no longer JP8.3, X3.3
- net N$35: now also JP8.9, X4.2; no longer JP8.2, X3.2
- net N$40: now also X9.7; no longer X8.7
- net N$42: now also X9.8; no longer X8.8
- net N$6: now also JP9.1, X5.8; no longer JP9.10, X4.8
- net N$60: now also SJ3.1; no longer SJ2.1
- net N$7: now also X9.2; no longer X8.2
- net N$75: now also X8.8; no longer X7.8
- net N$83: now also JP9.4, X5.5; no longer JP9.7, X4.5
- net N$84: now also JP9.9, X5.2; no longer JP9.2, X4.2
- net N$87: now also X8.1; no longer X7.1
- net N$9: now also X9.3; no longer X8.3
- net N$91: now also X8.2; no longer X7.2
- net N$93: now also X8.3; no longer X7.3
- net N$95: now also X8.4; no longer X7.4
- net N$97: now also X8.5; no longer X7.5
- net N$99: now also X8.6; no longer X7.6
- net RPOWA: now also SJ15.1, SJ17.1, SJ19.1; no longer SJ14.1, SJ16.1, SJ18.1
- net RPOWB: now also SJ16.1, SJ18.1, SJ20.1, X9.9; no longer SJ15.1, SJ17.1, SJ19.1, X8.9
- net SCK2: now also SJ2.1; no longer SJ20.1
- net SLNK1: now also SJ14.1; no longer SJ13.1
- net SLNK2: now also SJ5.1; no longer SJ4.1
- net SLNK3: now also SJ7.1; no longer SJ6.1
- net SRV5: now also G1.PC12; no longer G1.PF1-PH1
- net SRV7: now also G1.PF1-PH1; no longer G1.PC12
- net SW: now also D5.C, D6.C; no longer D3.C, D4.C
- net TOUT1: now also JP10.10, X7.1; no longer JP10.1, X6.1
- net TOUT2: now also JP10.9, X7.2; no longer JP10.2, X6.2
- net TOUT3: now also JP10.8, X7.3; no longer JP10.3, X6.3
- net TOUT4: now also JP10.7, X7.4; no longer JP10.4, X6.4
- net TOUT5: now also JP10.4, X7.5; no longer JP10.7, X6.5
- net TOUT6: now also JP10.3, X7.6; no longer JP10.8, X6.6
- net TOUT7: now also JP10.2, X7.7; no longer JP10.9, X6.7
- net TOUT8: now also JP10.1, X7.8; no longer JP10.10, X6.8
Other:
- note added: "Alternative population: Output ports D and E are optionally populated. If one output port is needed, populate port D (this sheet) and close SJ14. For options on populating U12, see sheet 6."
- note added: "Alternative population: Populate U6 and U9 to drive stall motor switch machines (e.g. Tortoise). This can also be used for CA or CC LED driving with appropriate external current limit resistors calculated for +15V. Multiple LEDs can be in series, too. Populate U5,7,8,10 with TC4426 or TC4427 to drive stall motors with more current needs in push-pull mode. Invert the output in software when switch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"
- note added: "Alternative population: This port is optionally populated. If not populated, close SJ14. For U13, may substitute 74HC595N if R3-R5 are populated. For HCT series those resistors are not necessary. For driving LEDs with up to 8 mA current, U14 may be populated with the series resistors for the LEDs directly. If external series resistors are present, the screw terminal can be soldered directly into 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"
- note added: "Close SJ7 if PORTB is not populated."
- note added: "Close both for F303RE."
- note added: "Close if 5V-DCDC switcher is not populated. Will use Nucleo's linear regulator from 12V to 5V, which has a strict current limit. Must observe max current consumption of the Nucleo specification, which depends on the input voltage. Putting any load by external peripherals is not recommended. Might work with lower voltage (e.g. 7V) input power."
- note added: "Close if U13 is missing."
- note added: "If SJ4 is closed, expn port SPI is parallel to onboard shift registers. If SJ4 is open and SJ5 is closed, they get daisy-chained."
- note added: "JP7: Power select jumper Bridge 1-2 and 3-4 in order to be bus powered (take power from OpenLCB bus). Bridge 1-3 and 2-4 in order to supply power to OpenLCB bus. Power plugged in to J1 is needed. Leave open in order to take power from power jack only. Power plugged in to J1 is needed."
- note added: "Populate R6-R13 if the servos in use are not compatible with 3V voltage levels. R6-R13: 5k-20k JP1-2 for SRV5-8 can not be populated if a Nucleo-144 board is used."
- note added: "Populate only one alternative - U2 (SOIC-8) with AP1509 and L1 with 47 uH inductor, or - U2B (PDIP-8) with LM2574N-5.0 and L1 with 470 uH inductor depending on the desired package."
- note added: "Populate only one alternative of U1 (PDIP-8) or U1B (SOIC-8) depending on the package. Example part choice: - MCP2551: R16 is 0 ohm or a slew control resistor. SJ18 open. - PCA82C250. R16 is 0 ohm or a slew control resistor. SJ18 open. - MCP2561, ATA6560/62: not recommended. - MCP2562 ATA6561/63: R16 is 0 ohm, SJ18 closed. - SN65HVD1050: R16 is 0 ohm, SJ18 open. - MCP2542FD: R16 is 0 ohm, SJ18 cl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"
- note added: "R1-R5: 5k-20k"
- note added: "Through-hole population: - populate RN2, RN4 with parallel resistor network or individual resistors. - populate RN1, RN3 with star resistor network. - do not populate R18-R49. SMD population: - populate R18-R49 - DNP RN1-4. Values: - RN2, RN4, R18-R25, R34-R41: 22k-270k. - RN1, RN3, R26-R33, R42-R49: 10k-270k."
- note added: "V+ is 5V power in to the Morpho connector 'E5V' pin. Will supply MCU with power via a linear regulator on the MCU board. The MCU board will connect it to the 5V output pin on the Morpho connector"
- note removed: "Alternative population: Output ports D and E are optionally populated. If one output port is needed, populate port D (this sheet) and close SJ17. For options on populating U14, see sheet 6."
- note removed: "Alternative population: Populate U9 and U10 to drive stall motor switch machines (e.g. Tortoise). This can also be used for CA or CC LED driving with appropriate external current limit resistors calculated for +15V. Multiple LEDs can be in series, too. Populate U3-U6 with TC4426 or TC4428 to drive high current (up to 1.5A per port) outputs in push-pull mode. Invert the output in software when swi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"
- note removed: "Alternative population: This port is optionally populated. If not populated, close SJ17. For U11, may substitute 74HC595N if R19-R21 are populated. For HCT series those resistors are not necessary. For driving LEDs with up to 8 mA current, U12 may be populated with the series resistors for the LEDs directly. If external series resistors are present, the screw terminal can be soldered directly int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"
- note removed: "Close S19 if PORTB is not populated."
- note removed: "Close for F303RE."
- note removed: "Close if 5V-DCDC switcher is not populated. Will use Nucleo's linear regulator from 12V to 5V, which produces a lot of heat; putting any load by external peripherals is not permissible. Might work with lower voltage (e.g. 7V) input power."
- note removed: "Close if U11 is missing."
- note removed: "If SJ15 is closed, expn port SPI is parallel to onboard shift registers. If SJ15 is open and SJ16 is closed, they get daisy-chained."
- note removed: "JP4: Power select jumper Bridge 1-2 and 3-4 in order to be bus powered (take power from OpenLCB bus). Bridge 1-3 and 2-4 in order to supply power to OpenLCB bus. Power plugged in to J3 is needed. Leave open in order to take power from power jack only. Power plugged in to J3 is needed."
- note removed: "Populate R24-27 and R64-67 if the servos in use are not compatible with 3V voltage levels. JP7-8 for SRV5-8 shall not be populated if a Nucleo-144 board is used."
- note removed: "Populate only one alternative - U8 (SOIC-8) with AP1509 or - U8B (PDIP-8) with LM2574N-5.0 depending on the desired package."
- note removed: "Populate only one alternative of U7 (PDIP-8) or U7B (SOIC-8) depending on the package. Example part choice: - MCP2551: R61 optional if slew rate control is needed. SJ18 open. - PCA82C250. R61 is 0 ohm or a slew control resistor. SJ18 open. - MCP2561, ATA6560/62: not recommended. - MCP2562 ATA6561/63: R61 is 0 ohm, SJ18 closed. - SN65HVD1050: R61 is 0 ohm, SJ18 open. - MCP2542FD: R61 is 0 ohm, SJ1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"
- note removed: "Through-hole population: - populate RN1, RN3 with parallel resistor network or individual resistors. - populate RN2, RN4 with star resistor network. - DNP R28-R60. SMD population: - populate R28-R60 - DNP RN1-4. Values: - RN1, RN3, R28-R44: 22k-270k. - RN2, RN4, R45-R60: 10k-270k."
- note removed: "V+ is 5V power in for the Morpho connector 'E5V' pin. Will supply MCU with power via a linear regulator on the MCU board. The MCU board will connect it to the 5V output pin on the Morpho connector"
- moved on the sheet: SJ10, SJ13, SJ14, SJ15, SJ16, SJ17, SJ2, SJ20, SJ5, SJ6, SJ7, SJ8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
