File: eagle/nucleo-io-board/io-board-d-8.brd (EAGLE design)
At the start: 100 x 80 mm, 169 parts, among them J1 DCJ0202, P1 9-15V DC, U1 CAN-TXR-PDIP, U10 TC4427, U11 74AHCT595N, U13 74AHCT595N, U1B CAN-TXR-SO8, U2 AP1509-50, U2B LM2574N-5.0, U3 74HC166, U4 74HC166, U5 TC4427, U6 LM324N, U7 TC4427, U8 TC4427, U9 LM324N, X1 RJ45-JACK, X2 RJ45-JACK, X4 M08-SCREW, X5 M09-SCREW, X7 M08-SCREW, X8 PORTD, X9 PORTE

Commit message: More versions of the board design.
Parts:
- removed D5: (no value), diode:DO41-7.6
- removed D6: DIODEDO-214AA-NODOC, trainlib:DO214AA-NODOC
- removed JP3: (no value), trainlib:JP3Q
- removed LG1: LCC_LOGO, tcs:LCC_LOGO
- removed LOGO1: DOC-OSHW-LOGOM, SPCoast:OSHW-LOGO-M
- removed SJ20: (no value), trainlib:SJ_RND2
- removed X7: M08-SCREW, trainlib:1X08_TERMINAL
- removed X8: PORTD, trainlib:1X09_TERMINAL
- removed X9: PORTE, trainlib:1X09_TERMINAL
- added J2: RJ45-JACK, trainlib:RJ45-PULSE-E5J88
- added J3: DCJ0202, con-jack:DCJ0202
- added J4: (no value), con-jack:SPC4077
- added PORTB: (no value), trainlib:CON10M
- C2: device rcl:C1206 -> rcl:E2,5-5
- C5: device rcl:C1206 -> rcl:C0805
- C6: device rcl:E2,5-5 -> rcl:C1206
- C8: device rcl:C0805 -> rcl:C1206
- D1: value DIODEDO-214AA-NODOC -> (none); device trainlib:DO214AA-NODOC -> diode:DO41-7.6
- D4: value (none) -> DIODEDO-214AA-NODOC; device diode:DO41-7.6 -> trainlib:DO214AA-NODOC
- J1: value DCJ0202 -> RJ45-JACK; device trainlib:DCJ0202 -> trainlib:RJ45-PULSE-E5J88
- JP1: device trainlib:JP3Q -> trainlib:JP4F
- JP2: value (none) -> JP8-FLAT; device trainlib:JP3Q -> trainlib:JP8F
- JP4: device trainlib:JP3Q -> trainlib:JP2Q
- JP5: value JP8-FLATFEMALE -> (none); device trainlib:JP8F-FEM -> trainlib:JP3Q
- JP6: device trainlib:JP4F -> trainlib:JP3Q
- JP7: device trainlib:JP2Q -> trainlib:JP3Q
- JP8: value PORTB -> (none); device trainlib:CON10M -> trainlib:JP3Q
- PORTA: value PORTA -> (none)
- PORTC: value PORTC -> (none)
- R1, R2: value (none) -> 10k
- R10, R11, R12, R13, R16, R3, R4, R5, R6, R7, R8, R9: device rcl:R0805 -> rcl:R0603
- R14, R15: value 5k -> (none); device rcl:R0805 -> rcl:R0603
- R17: value 500mA -> (none); device tcs:PTC1812 -> rcl:R0603
- R19, R20, R21, R22, R23, R24, R25, R61, R62, R63, R64, R65, R66, R67: device rcl:R0603 -> rcl:R0805
- R26, R27: device trainlib:R0603 -> rcl:R0805
- R28, R29, R30, R31, R32, R33, R42, R43, R44: device trainlib:R0603 -> rcl:R0603
- R40: value (none) -> 500mA; device rcl:R0603 -> tcs:PTC1812
- R50, R51: value 10k -> (none); device rcl:R0805 -> trainlib:R0603
- R52, R53, R54, R55, R56, R57, R58, R59, R60: device rcl:R0603 -> trainlib:R0603
- RN1, RN3: value 10K -> (none); device resistor-sil:SIL9 -> resistor-dil:DIL16
- RN2, RN4: value (none) -> 10K; device resistor-dil:DIL16 -> resistor-sil:SIL9
- SJ12, SJ19, SJ4: device trainlib:SJW-C -> trainlib:SJ_RND2
- SJ15, SJ3, SJ9: device trainlib:SJ_RND2 -> trainlib:SJW-C
- U1: value CAN-TXR-PDIP -> 74HC166; device trainlib:DIL08 -> 74xx-us:DIL16
- U10: value TC4427 -> LM324N; device trainlib:DIL08-LONG -> linear:DIL14
- U11, U13: device trainlib:DIL16 -> 74xx-eu:DIL16
- U2: value AP1509-50 -> 74HC166; device trainlib:SO-08 -> 74xx-us:DIL16
- U3, U4: value 74HC166 -> TC4426/28; device trainlib:DIL16 -> trainlib:DIL08-LONG
- U5: value TC4427 -> TC4426/28
- U6: value LM324N -> TC4426/28; device trainlib:DIL14 -> trainlib:DIL08-LONG
- U7: value TC4427 -> CAN-TXR-PDIP; device trainlib:DIL08-LONG -> trainlib:DIL08
- U8: value TC4427 -> AP1509-50; device trainlib:DIL08-LONG -> trainlib:SO-08
- U9: device trainlib:DIL14 -> linear:DIL14
- X1, X2: value RJ45-JACK -> M08-SCREW; device trainlib:RJ45-PULSE-E5J88 -> trainlib:1X08_TERMINAL
- X3: value (none) -> M08-SCREW; device SPCoast:SCREWTERMINAL-3.5MM-2_LOCK -> trainlib:1X08_TERMINAL
- X4: value M08-SCREW -> PORTD
- X5: value M09-SCREW -> PORTE; device trainlib:1X09_TERMINAL -> trainlib:1X08_TERMINAL
- moved JP4 106.4 mm to (88.4, 3.56), turned to 0 degrees
- moved C2 104.6 mm to (97.8, 68.6), turned to 270 degrees
- moved X1 101.4 mm to (3.10, 70.4), turned to 270 degrees
- moved X3 94.6 mm to (3.10, 27.6), turned to 270 degrees
- moved X2 92.2 mm to (3.10, 49.0), turned to 270 degrees
- moved X5 86.1 mm to (55.9, 3.10), turned to 0 degrees
- moved R63 83.2 mm to (18.5, 77.7), turned to 0 degrees
- moved R62 83.2 mm to (18.5, 75.8), flipped to the top, turned to 0 degrees
- moved JP2 81.3 mm to (66.0, 69.8), turned to 0 degrees
- moved C6 80.9 mm to (25.9, 31.5), turned to 0 degrees
- moved R13 78.9 mm to (36.8, 9.40), turned to 90 degrees
- moved R12 77.2 mm to (34.3, 9.40), flipped to the bottom, turned to 90 degrees
- moved C1 75.6 mm to (90.7, 77.0)
- moved R40 74.5 mm to (80.0, 5.08), turned to 90 degrees
- moved C7 71.7 mm to (35.3, 31.5), turned to 180 degrees
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- renumbered G1 to U$1, JP10 to PORTC, JP9 to PORTA, P1 to +12V, U1B to U7B, U2B to U8B
Connections:
- removed net ALT1: X1.4, X2.4
- removed net ALT2: X1.5, X2.5
- removed net SCK2_ALT: SJ2.P$2, U$1.PB13
- new net N$36: PORTB.1, R35.2, R45.2, RN1.1, RN2.9, X2.1
- net +12V: now also C6.1, C7.1, J3.1, JP2.7, JP4.2, SJ14.P$2, SJ2.P$2, SJ5.P$2, SJ8.P$2, U10.4, U3.6, U4.6, U6.6, U8.1; no longer C5.1, C9.1, D3.C, D4.C, JP5.7, JP7.2, SJ10.P$2, SJ17.P$2, SJ18.P$2, SJ3.P$2, U10.6, U2.1, U6.4, U7.6, U8.6
- net +3V3: now also C11.1, R1.2, R50.1, R51.1, R52.1, R53.1, R54.1, R55.1, R56.1, R57.1, R58.1, R59.1, R60.1, RN2.1, RN4.1, SJ18.P$1, U1.1, U1.16, U1.9, U2.16, U2.9; no longer C8.1, R26.1, R27.1, R28.1, R29.1, R30.1, R31.1, R32.1, R33.1, R42.1, R43.1, R44.1, R50.2, RN1.1, RN3.1, SJ6.P$1, U3.16, U3.9, U4.1, U4.16, U4.9
- net +5V: now also C5.1, C8.1, C9.1, JP2.6, JP5.3, JP5.4, JP6.4, JP7.3, JP7.4, JP8.3, JP8.4, PORTB.6, R19.2, R20.2, R21.2, R22.1, R23.1, R24.1, R25.1, R26.1, R27.1, R62.1, R63.1, R64.1, R65.1, R66.1, R67.1, SJ1.P$2, SJ10.P$2, SJ4.P$2, SJ7.P$2, U7.3; no longer C1.1, C11.1, C2.1, JP1.4, JP2.3, JP2.4, JP3.3, JP3.4, JP4.3, JP4.4, JP5.6, JP8.6, R1.1, R10.1, R11.1, R12.1, R13.1, R14.1, R15.1, R2.1, R3.2, R4.2, R5.2, R6.1, R7.1, R8.1, R9.1, SJ15.P$2, SJ16.P$2, SJ8.P$2, SJ9.P$2, U1.3
- net CANH: now also J1.1, J2.1, U7.7; no longer U1.7, X1.1, X2.1
- net CANL: now also J1.2, J2.2, U7.6; no longer U1.6, X1.2, X2.2
- net CANRX: now also U7.4; no longer U1.4
- net CANTX: now also U7.1; no longer U1.1
- net CAN_RS: now also R61.1, U7.8; no longer R16.1, U1.8
- net CAN_VIO: now also SJ18.P$2, U7.5; no longer SJ6.P$2, U1.5
- net CMPREF: now also R1.1, R2.2, U10.13, U10.2, U10.6, U10.9; no longer R50.1, R51.2, U6.13, U6.2, U6.6, U6.9
- net E_CS: now also JP2.4, R23.2; no longer JP5.4, R1.2
- net E_LAT: now also JP2.5, R22.2; no longer JP5.5, R2.2
- net E_MOSI: now also JP2.2, SJ15.2, SJ16.P$2; no longer JP5.2, SJ4.2, SJ5.P$2
- net GND: now also C2.-, C6.2, D1.A, D3.A, J1.6, J1.7, J2.3, J2.6, J2.7, J3.2, J3.3, JP1.4, JP2.8, JP5.5, JP5.6, JP6.5, JP6.6, JP7.5, JP7.6, JP8.6, PORTB.5, R2.1, R61.2, SJ12.P$2, SJ3.2, SJ6.P$2, SJ9.2, U1.6, U1.8, U10.11, U3.3, U4.3, U6.3, U7.2, U8.4, U8.5, U8.6, U8.7, U8.8; no longer C2.2, C6.-, D5.A, D6.A, J1.2, J1.2B, J1.3B, JP1.5, JP1.6, JP2.5, JP2.6, JP3.5, JP3.6, JP4.5, JP4.6, JP5.8, JP6.4, R16.2, R51.1, SJ12.2, SJ13.P$2, SJ19.2, SJ20.P$2, U1.2, U10.3, U2.4, U2.5, U2.7, U3.6, U3.8, U4.6, U4.8, U6.11, U7.3, U8.3, X1.3, X1.6, X1.7, X2.3, X2.6, X2.7, X3.2, X5.9
- net I2CSCL: now also JP1.1, R62.2; no longer JP6.1, R15.2
- net I2CSDA: now also JP1.2, R63.2; no longer JP6.2, R14.2
- net ILAT: now also U1.15, U2.15; no longer U3.15, U4.15
- net LPOWA: now also SJ7.P$1, SJ9.1, U14.9; no longer SJ10.P$1, SJ12.1, U12.9
- net LPOWB: now also SJ10.P$1, SJ12.P$1, U14.10; no longer SJ13.P$1, SJ9.P$1, U12.10, X8.9
- net MISO: now also JP2.1; no longer JP5.1
- net MISO2: now also SJ13.P$2, SJ19.P$2, U2.13; no longer SJ1.P$2, SJ7.P$2, U3.13
- net MISO2_ALT: now also SJ13.P$1; no longer SJ1.P$1
- net MOSI: now also R20.1, SJ15.1, SJ17.P$2, U11.14; no longer R4.1, SJ14.P$2, SJ4.1, U13.14
- net N$1: now also R3.1, U11.15, U12.1; no longer R67.1, U13.15, U14.1
- net N$10: now also R6.1, U11.3, U12.4; no longer R64.1, U13.3, U14.4
- net N$100: now also R17.1, U13.6, U14.7; no longer R53.1, U11.6, U12.7
- net N$101: now also Q15.3, U14.12, X4.7; no longer Q2.3, U12.12, X8.7
- net N$102: now also R18.1, U13.7, U14.8; no longer R52.1, U11.7, U12.8
- net N$104: now also Q9.1, R11.2; no longer Q8.1, R59.2
- net N$105: now also Q10.1, R12.2; no longer Q7.1, R58.2
- net N$106: now also Q11.1, R13.2; no longer Q6.1, R57.2
- net N$107: now also Q12.1, R14.2; no longer Q5.1, R56.2
- net N$108: now also Q13.1, R15.2; no longer Q4.1, R55.2
- net N$109: now also Q14.1, R16.2; no longer Q3.1, R54.2
- net N$11: now also Q4.3, U12.15, X5.4; no longer Q13.3, U14.15, X9.4
- net N$110: now also Q15.1, R17.2; no longer Q2.1, R53.2
- net N$111: now also Q16.1, R18.2; no longer Q1.1, R52.2
- net N$12: now also R7.1, U11.4, U12.5; no longer R63.1, U13.4, U14.5
- net N$13: now also Q5.3, U12.14, X5.5; no longer Q12.3, U14.14, X9.5
- net N$14: now also PORTA.9, R37.2, R59.2, RN3.7, RN4.3, X1.7; no longer PORTA.2, R35.2, R48.2, RN3.3, RN4.7, X5.7
- net N$15: now also PORTA.8, R38.2, R58.2, RN3.6, RN4.4, X1.6; no longer PORTA.3, R36.2, R47.2, RN3.4, RN4.6, X5.6
- net N$16: now also Q4.1, R6.2; no longer Q13.1, R64.2
- net N$17: now also R8.1, U11.5, U12.6; no longer R62.1, U13.5, U14.6
- net N$18: now also Q6.3, U12.13, X5.6; no longer Q11.3, U14.13, X9.6
- net N$19: now also PORTA.4, R41.2, R56.2, RN3.4, RN4.6, X1.4; no longer PORTA.7, R38.2, R45.2, RN3.6, RN4.4, X5.4
- net N$2: now also Q1.3, U12.18, X5.1; no longer Q16.3, U14.18, X9.1
- net N$20: now also PORTA.3, R42.2, R55.2, RN3.3, RN4.7, X1.3; no longer PORTA.8, R39.2, R44.2, RN3.7, RN4.3, X5.3
- net N$21: now also PORTB.8, R30.2, R50.2, RN1.6, RN2.4, X2.6; no longer JP8.3, R20.2, R31.2, RN1.4, RN2.6, X4.6
- net N$22: now also PORTA.1, R44.2, R53.2, RN3.1, RN4.9, X1.1; no longer PORTA.10, R41.2, R42.2, RN3.9, RN4.1, X5.1
- net N$23: now also R36.1, RN3.9, U1.2; no longer R34.1, RN4.9, U4.2
- net N$24: now also R37.1, RN3.10, U1.3; no longer R35.1, RN4.10, U4.3
- net N$25: now also PORTB.10, R28.2, R52.2, RN1.8, RN2.2, X2.8; no longer JP8.1, R18.2, R33.2, RN1.2, RN2.8, X4.8
- net N$26: now also PORTB.9, R29.2, R51.2, RN1.7, RN2.3, X2.7; no longer JP8.2, R19.2, R32.2, RN1.3, RN2.7, X4.7
- net N$27: now also Q5.1, R7.2; no longer Q12.1, R63.2
- net N$28: now also PORTB.7, R31.2, R49.2, X2.5; no longer JP8.4, R21.2, R30.2, X4.5
- net N$29: now also R38.1, RN3.11, U1.4; no longer R36.1, RN4.11, U4.4
- net N$3: now also R4.1, U11.1, U12.2; no longer R66.1, U13.1, U14.2
- net N$30: now also R39.1, RN3.12, U1.5; no longer R37.1, RN4.12, U4.5
- net N$31: now also R41.1, RN3.13, U1.10; no longer R38.1, RN4.13, U4.10
- net N$32: now also R42.1, RN3.14, U1.11; no longer R39.1, RN4.14, U4.11
- net N$33: now also PORTB.4, R32.2, R48.2, RN1.4, RN2.6, X2.4; no longer JP8.7, R22.2, R29.2, RN1.6, RN2.4, X4.4
- net N$34: now also PORTB.3, R33.2, R47.2, RN1.3, RN2.7, X2.3; no longer JP8.8, R23.2, R28.2, RN1.7, RN2.3, X4.3
- net N$35: now also PORTB.2, R34.2, R46.2, RN1.2, RN2.8, X2.2; no longer JP8.9, R24.2, R27.2, RN1.8, RN2.2, X4.2
- net N$37: now also R43.1, RN3.15, U1.12; no longer R40.1, RN4.15, U4.12
- net N$38: now also R44.1, RN3.16, U1.14; no longer R41.1, RN4.16, U4.14
- net N$39: now also R9.1, U11.6, U12.7; no longer R61.1, U13.6, U14.7
- net N$4: now also J1.4, J2.4; no longer D3.A, D4.A, J1.1, J1.1B, X3.1
- net N$40: now also Q7.3, U12.12, X5.7; no longer Q10.3, U14.12, X9.7
- net N$41: now also R10.1, U11.7, U12.8; no longer R60.1, U13.7, U14.8
- net N$42: now also Q8.3, U12.11, X5.8; no longer Q9.3, U14.11, X9.8
- net N$43: now also Q6.1, R8.2; no longer Q11.1, R62.2
- net N$44: now also R28.1, RN1.9, U2.2; no longer R18.1, RN2.9, U3.2
- net N$45: now also D4.C, JP4.1; no longer D1.C, JP7.1
- net N$46: now also D4.A, JP4.4; no longer D1.A, JP7.4
- net N$47: now also R29.1, RN1.10, U2.3; no longer R19.1, RN2.10, U3.3
- net N$48: now also R30.1, RN1.11, U2.4; no longer R20.1, RN2.11, U3.4
- net N$49: now also R31.1, RN1.12, U2.5; no longer R21.1, RN2.12, U3.5
- net N$5: now also J1.5, J2.5; no longer JP8.10, R25.2, R26.2, RN1.9, RN2.1, X4.1
- net N$50: now also R32.1, RN1.13, U2.10; no longer R22.1, RN2.13, U3.10
- net N$51: now also R33.1, RN1.14, U2.11; no longer R23.1, RN2.14, U3.11
- net N$52: now also R34.1, RN1.15, U2.12; no longer R24.1, RN2.15, U3.12
- net N$53: now also R35.1, RN1.16, U2.14; no longer R25.1, RN2.16, U3.14
- net N$56: now also R11.1, U13.15, U14.1; no longer R59.1, U11.15, U12.1
- net N$57: now also JP4.3, R40.1; no longer JP7.3, R17.1
- net N$6: now also PORTA.10, R36.2, R60.2, RN3.8, RN4.2, X1.8; no longer PORTA.1, R34.2, R49.2, RN3.2, RN4.8, X5.8
- net N$60: now also SJ14.P$1; no longer SJ3.P$1
- net N$65: now also Q7.1, R9.2; no longer Q10.1, R61.2
- net N$7: now also Q2.3, U12.17, X5.2; no longer Q15.3, U14.17, X9.2
- net N$75: now also Q16.3, U14.11, X4.8; no longer Q1.3, U12.11, X8.8
- net N$78: now also Q1.1, R3.2; no longer Q16.1, R67.2
- net N$79: now also Q2.1, R4.2; no longer Q15.1, R66.2
- net N$8: now also R5.1, U11.2, U12.3; no longer R65.1, U13.2, U14.3
- net N$83: now also PORTA.7, R39.2, R57.2, X1.5; no longer PORTA.4, R37.2, R46.2, X5.5
- net N$84: now also PORTA.2, R54.2, RN3.2, RN4.8, X1.2; no longer PORTA.9, R40.2, RN3.8, RN4.2, X5.2
- net N$85: now also Q8.1, R10.2; no longer Q9.1, R60.2
- net N$87: now also Q9.3, U14.18, X4.1; no longer Q8.3, U12.18, X8.1
- net N$88: now also Q3.1, R5.2; no longer Q14.1, R65.2
- net N$89: now also R12.1, U13.1, U14.2; no longer R58.1, U11.1, U12.2
- net N$9: now also Q3.3, U12.16, X5.3; no longer Q14.3, U14.16, X9.3
- net N$91: now also Q10.3, U14.17, X4.2; no longer Q7.3, U12.17, X8.2
- net N$92: now also R13.1, U13.2, U14.3; no longer R57.1, U11.2, U12.3
- net N$93: now also Q11.3, U14.16, X4.3; no longer Q6.3, U12.16, X8.3
- net N$94: now also R14.1, U13.3, U14.4; no longer R56.1, U11.3, U12.4
- net N$95: now also Q12.3, U14.15, X4.4; no longer Q5.3, U12.15, X8.4
- net N$96: now also R15.1, U13.4, U14.5; no longer R55.1, U11.4, U12.5
- net N$97: now also Q13.3, U14.14, X4.5; no longer Q4.3, U12.14, X8.5
- net N$98: now also R16.1, U13.5, U14.6; no longer R54.1, U11.5, U12.6
- net N$99: now also Q14.3, U14.13, X4.6; no longer Q3.3, U12.13, X8.6
- net OLAT: now also R21.1; no longer R3.1
- net PWR_POS: now also J1.8, J2.8, R40.2; no longer R17.2, X1.8, X2.8
- net RPOWA: now also SJ1.P$1, SJ2.P$1, SJ3.1, U12.9; no longer SJ15.P$1, SJ17.P$1, SJ19.1, U14.9
- net RPOWB: now also SJ4.P$1, SJ5.P$1, SJ6.P$1, U12.10; no longer SJ16.P$1, SJ18.P$1, SJ20.P$1, U14.10, X9.9
- net SCK: now also JP2.3, R19.1; no longer JP5.3, R5.1
- net SCK2: now also U1.7, U2.7; no longer SJ2.P$1, U3.7, U4.7
- net SLNK1: now also SJ17.P$1, U11.9, U13.14; no longer SJ14.P$1, U11.14, U13.9
- net SLNK2: now also SJ16.P$1, U13.9; no longer SJ5.P$1, U11.9
- net SLNK3: now also SJ19.P$1, U1.13, U2.1; no longer SJ7.P$1, U3.1, U4.13
- net SRV1: now also JP5.2, R24.2; no longer JP4.2, R13.2
- net SRV2: now also JP5.1, R25.2; no longer JP4.1, R12.2
- net SRV3: now also JP6.2, R26.2; no longer JP3.2, R11.2
- net SRV4: now also JP6.1, R27.2; no longer JP3.1, R10.2
- net SRV5: now also JP7.2, R64.2, U$1.PF1-PH1; no longer JP2.2, R9.2, U$1.PC12
- net SRV6: now also JP7.1, R65.2; no longer JP2.1, R8.2
- net SRV7: now also JP8.2, R66.2, U$1.PC12; no longer JP1.2, R7.2, U$1.PF1-PH1
- net SRV8: now also JP8.1, R67.2; no longer JP1.1, R6.2
- net SW: now also D1.C, D3.C, U8.2; no longer D5.C, D6.C, U2.2
- net TDRV1: now also U10.12, U6.2; no longer U10.2, U9.12
- net TDRV2: now also U10.3, U6.4; no longer U10.4, U9.3
- net TDRV3: now also U10.10, U5.4; no longer U8.4, U9.10
- net TDRV4: now also U10.5, U5.2; no longer U8.2, U9.5
- net TDRV5: now also U4.2, U9.12; no longer U6.12, U7.2
- net TDRV6: now also U4.4, U9.3; no longer U6.3, U7.4
- net TDRV7: now also U3.4, U9.10; no longer U5.4, U6.10
- net TDRV8: now also U3.2, U9.5; no longer U5.2, U6.5
- net TOUT1: now also PORTC.1, U3.7, U9.7, X3.1; no longer PORTC.10, U5.7, U6.7, X7.1
- net TOUT2: now also PORTC.2, U3.5, U9.8, X3.2; no longer PORTC.9, U5.5, U6.8, X7.2
- net TOUT3: now also PORTC.3, U4.5, U9.1, X3.3; no longer PORTC.8, U6.1, U7.5, X7.3
- net TOUT4: now also PORTC.4, U4.7, U9.14, X3.4; no longer PORTC.7, U6.14, U7.7, X7.4
- net TOUT5: now also PORTC.7, U10.7, U5.7, X3.5; no longer PORTC.4, U8.7, U9.7, X7.5
- net TOUT6: now also PORTC.8, U10.8, U5.5, X3.6; no longer PORTC.3, U8.5, U9.8, X7.6
- net TOUT7: now also PORTC.9, U10.1, U6.5, X3.7; no longer PORTC.2, U10.5, U9.1, X7.7
- net TOUT8: now also PORTC.10, U10.14, U6.7, X3.8; no longer PORTC.1, U10.7, U9.14, X7.8
- net V+: now also C1.1, C2.+, U8.3; no longer C6.+, C7.1, U2.3
Routing:
- net N$36: track 0.00 -> 79.7 mm
- net SRV7: track 38.5 -> 116.9 mm, vias 2 -> 3
- net SRV5: track 104.1 -> 40.3 mm
- net N$5: track 79.3 -> 20.9 mm
- net ALT2: track 24.2 -> 0.00 mm, vias 1 -> 0
- net ALT1: track 20.5 -> 0.00 mm, vias 1 -> 0
- net GND: track 758.9 -> 774.1 mm, vias 224 -> 203
- net RPOWB: track 25.3 -> 11.8 mm
- net LPOWB: track 44.3 -> 31.7 mm
- net +5V: track 441.0 -> 430.4 mm, vias 15 -> 17
- net PWR_POS: track 47.0 -> 57.0 mm, vias 1 -> 0
- net +12V: track 276.1 -> 268.6 mm
- net SCK2: track 62.5 -> 55.1 mm
- net CANL: track 112.9 -> 118.4 mm, vias 5 -> 6
- net CANH: track 118.2 -> 122.4 mm, vias 5 -> 6
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Other:
- board text added: "JP4: PWR =OUT || IN :: LOC"
- board text removed: "100"
- board text removed: "500"
- board text removed: "GND 12V"
- board text removed: "JP7: PWR =OUT :: LOCL || IN"
- board text removed: "OpenLCB Dev IO Rev. B. 2018-05-06"
