File: eagle/nucleo-io-board/io-board-d-8.sch (EAGLE design)
At the start: 169 parts, among them J1 DCJ0202, P1 9-15V DC, Q1 BSS123, Q10 BSS123, Q11 BSS123, Q12 BSS123, Q13 BSS123, Q14 BSS123, Q15 BSS123, Q16 BSS123, Q2 BSS123, Q3 BSS123, Q4 BSS123, Q5 BSS123, Q6 BSS123, Q7 BSS123, Q8 BSS123, Q9 BSS123, U1 CAN-TXR-PDIP, U10 TC4427, U11 74AHCT595N, U13 74AHCT595N, U1B CAN-TXR-SO8, U2 AP1509-50, U2B LM2574N-5.0, U3 74HC166, U4 74HC166, U5 TC4427, U6 LM324N, U7 TC4427, U8 TC4427, U9 LM324N, X1 RJ45-JACK, X2 RJ45-JACK, X4 M08-SCREW, X5 M09-SCREW, X7 M08-SCREW, X8 PORTD, X9 PORTE

Commit message: More versions of the board design.
Parts:
- removed D5: (no value), diode:DIODE-DO41-7.6
- removed D6: DIODEDO-214AA-NODOC, trainlib:DIODEDO-214AA-NODOC
- removed JP10: PORTC, trainlib:PINHD-2X5CN
- removed JP3: (no value), trainlib:JP3Q
- removed JP9: PORTA, trainlib:PINHD-2X5CN
- removed LG1: LCC_LOGO, tcs:LCC_LOGO
- removed LOGO1: DOC-OSHW-LOGOM, SPCoast:DOC-OSHW-LOGOM
- removed P1: 9-15V DC, SPCoast:DOC-POWER_LABEL
- removed SJ20: (no value), trainlib:SJRND2
- removed U1B: CAN-TXR-SO8, SPCoast:MCP2551-SN
- removed U2B: LM2574N-5.0, linear:LM2574N-5.0
- removed X7: M08-SCREW, trainlib:M08-SCREW
- removed X8: PORTD, trainlib:M09-SCREW
- removed X9: PORTE, trainlib:M09-SCREW
- added +12V: 9-15V DC, SPCoast:DOC-POWER_LABEL
- added J2: RJ45-JACK, trainlib:RJ45-JACKRJ45-PULSE-E5J00
- added J3: DCJ0202, con-jack:DCJ0202
- added J4: (no value), con-jack:JACK-PLUG0
- added PORTA, PORTB, PORTC: (no value), trainlib:PINHD-2X5CN
- added U7B: CAN-TXR-SO8, SPCoast:MCP2551-SN
- added U8B: LM2574N-5.0, linear:LM2574N-5.0
- C1, C10: device rcl:C-USC1206 -> rcl:C-EUC1206
- C2: device rcl:C-USC1206 -> rcl:CPOL-USE2.5-5
- C5: device rcl:C-EUC1206 -> rcl:C-USC0805
- C6: device rcl:CPOL-USE2.5-5 -> rcl:C-USC1206
- C7: device rcl:C-EUC1206 -> rcl:C-USC1206
- C8: device rcl:C-USC0805 -> rcl:C-USC1206
- D1: value DIODEDO-214AA-NODOC -> (none); device trainlib:DIODEDO-214AA-NODOC -> diode:DIODE-DO41-7.6
- D4: value (none) -> DIODEDO-214AA-NODOC; device diode:DIODE-DO41-7.6 -> trainlib:DIODEDO-214AA-NODOC
- J1: value DCJ0202 -> RJ45-JACK; device trainlib:DCJ0202 -> trainlib:RJ45-JACKRJ45-PULSE-E5J00
- JP1: device trainlib:JP3Q -> trainlib:JP4-FLAT
- JP2: value (none) -> JP8-FLAT; device trainlib:JP3Q -> trainlib:JP8-FLAT
- JP4: device trainlib:JP3Q -> trainlib:JP2Q
- JP5: value JP8-FLATFEMALE -> (none); device trainlib:JP8-FLATFEMALE -> trainlib:JP3Q
- JP6: device trainlib:JP4-FLAT -> trainlib:JP3Q
- JP7: device trainlib:JP2Q -> trainlib:JP3Q
- JP8: value PORTB -> (none); device trainlib:PINHD-2X5CN -> trainlib:JP3Q
- R1, R2: value (none) -> 10k
- R10, R11, R12, R13, R16, R3, R4, R5, R6, R7, R8, R9: device rcl:R-US_R0805 -> rcl:R-US_R0603
- R14, R15: value 5k -> (none); device rcl:R-US_R0805 -> rcl:R-US_R0603
- R17: value 500mA -> (none); device tcs:PTC_1812 -> rcl:R-US_R0603
- R19, R20, R21, R22, R23, R24, R25, R61, R62, R63, R64, R65, R66, R67: device rcl:R-US_R0603 -> rcl:R-US_R0805
- R26, R27: value R-US -> (none); device trainlib:R-US -> rcl:R-US_R0805
- R28, R29, R30, R31, R32, R33, R42, R43, R44: value R-US -> (none); device trainlib:R-US -> rcl:R-US_R0603
- R40: value (none) -> 500mA; device rcl:R-US_R0603 -> tcs:PTC_1812
- R50, R51: value 10k -> R-US; device rcl:R-US_R0805 -> trainlib:R-US
- R52, R53, R54, R55, R56, R57, R58, R59, R60: value (none) -> R-US; device rcl:R-US_R0603 -> trainlib:R-US
- RN1, RN3: value 10K -> (none); device resistor-sil:G08R -> resistor-dil:8R-P
- RN2, RN4: value (none) -> 10K; device resistor-dil:8R-P -> resistor-sil:G08R
- SJ12, SJ19, SJ4: device trainlib:SJ-C -> trainlib:SJRND2
- SJ15, SJ3, SJ9: device trainlib:SJRND2 -> trainlib:SJ-C
- U1: value CAN-TXR-PDIP -> 74HC166; device trainlib:PCA82C250 -> 74xx-us:74166N
- U10: value TC4427 -> LM324N; device trainlib:TC4426APDIP -> linear:LM324N
- U11, U13: device trainlib:74HCT595N -> 74xx-eu:74HCT595N
- U2: value AP1509-50 -> 74HC166; device trainlib:AP1509 -> 74xx-us:74166N
- U3, U4: value 74HC166 -> TC4426/28; device trainlib:74166N -> trainlib:TC4426APDIP
- U5: value TC4427 -> TC4426/28
- U6: value LM324N -> TC4426/28; device trainlib:LM324N -> trainlib:TC4426APDIP
- U7: value TC4427 -> CAN-TXR-PDIP; device trainlib:TC4426APDIP -> trainlib:PCA82C250
- U8: value TC4427 -> AP1509-50; device trainlib:TC4426APDIP -> trainlib:AP1509
- U9: device trainlib:LM324N -> linear:LM324N
- X1, X2: value RJ45-JACK -> M08-SCREW; device trainlib:RJ45-JACKRJ45-PULSE-E5J00 -> trainlib:M08-SCREW
- X3: value (none) -> M08-SCREW; device SPCoast:CONNECTOR-M023.5MM-LOCK -> trainlib:M08-SCREW
- X4: value M08-SCREW -> PORTD
- X5: value M09-SCREW -> PORTE; device trainlib:M09-SCREW -> trainlib:M08-SCREW
- renumbered G1 to U$1
Connections:
- removed net ALT1: X1.4, X2.4
- removed net ALT2: X1.5, X2.5
- removed net SCK2_ALT: SJ2.2, U$1.PB13
- new net N$36: PORTB.1, R35.2, R45.2, RN1A.1, RN2.9, X2.1
- net +12V: now also C6.1, C7.1, J3.1, JP2.7, JP4.2, SJ14.2, SJ2.2, SJ5.2, SJ8.2, U10P.V+, U3P.VDD, U4P.VDD, U6P.VDD, U8.VIN, U8B.IN; no longer C5.1, C9.1, D3.C, D4.C, JP5.7, JP7.2, SJ10.2, SJ17.2, SJ18.2, SJ3.2, U10P.VDD, U2.VIN, U2B.IN, U6P.V+, U7P.VDD, U8P.VDD
- net +3V3: now also C11.1, R1.2, R50.1, R51.1, R52.1, R53.1, R54.1, R55.1, R56.1, R57.1, R58.1, R59.1, R60.1, RN2.1, RN4.1, SJ18.1, U1A.CLR, U1A.SER, U1P.VCC, U2A.CLR, U2P.VCC; no longer C8.1, R26.1, R27.1, R28.1, R29.1, R30.1, R31.1, R32.1, R33.1, R42.1, R43.1, R44.1, R50.2, RN1.1, RN3.1, SJ6.1, U3A.CLR, U3P.VCC, U4A.CLR, U4A.SER, U4P.VCC
- net +5V: now also C5.1, C8.1, C9.1, JP2.6, JP5.3, JP5.4, JP6.4, JP7.3, JP7.4, JP8.3, JP8.4, PORTA.6, PORTB.6, PORTC.6, R19.2, R20.2, R21.2, R22.1, R23.1, R24.1, R25.1, R26.1, R27.1, R62.1, R63.1, R64.1, R65.1, R66.1, R67.1, SJ1.2, SJ10.2, SJ4.2, SJ7.2, U7.VCC, U7B.VDD; no longer C1.1, C11.1, C2.1, JP1.4, JP10.6, JP2.3, JP2.4, JP3.3, JP3.4, JP4.3, JP4.4, JP5.6, JP8.6, JP9.6, R1.1, R10.1, R11.1, R12.1, R13.1, R14.1, R15.1, R2.1, R3.2, R4.2, R5.2, R6.1, R7.1, R8.1, R9.1, SJ15.2, SJ16.2, SJ8.2, SJ9.2, U1.VCC, U1B.VDD
- net CANH: now also J1.1, J2.1, U7.CANH, U7B.CANH; no longer U1.CANH, U1B.CANH, X1.1, X2.1
- net CANL: now also J1.2, J2.2, U7.CANL, U7B.CANL; no longer U1.CANL, U1B.CANL, X1.2, X2.2
- net CANRX: now also U7.RXD, U7B.RXD; no longer U1.RXD, U1B.RXD
- net CANTX: now also U7.TXD, U7B.TXD; no longer U1.TXD, U1B.TXD
- net CAN_RS: now also R61.1, U7.RS, U7B.RS; no longer R16.1, U1.RS, U1B.RS
- net CAN_VIO: now also SJ18.2, U7.VREF, U7B.VREF; no longer SJ6.2, U1.VREF, U1B.VREF
- net CMPREF: now also R1.1, R2.2, U10A.-IN, U10B.-IN, U10C.-IN, U10D.-IN; no longer R50.1, R51.2, U6A.-IN, U6B.-IN, U6C.-IN, U6D.-IN
- net E_CS: now also JP2.4, R23.2; no longer JP5.4, R1.2
- net E_LAT: now also JP2.5, R22.2; no longer JP5.5, R2.2
- net E_MOSI: now also JP2.2, SJ15.2, SJ16.2; no longer JP5.2, SJ4.2, SJ5.2
- net GND: now also C2.-, C6.2, D1.A, D3.A, J1.6, J1.7, J2.3, J2.6, J2.7, J3.2, J3.3, JP1.4, JP2.8, JP5.5, JP5.6, JP6.5, JP6.6, JP7.5, JP7.6, JP8.6, PORTA.5, PORTB.5, PORTC.5, R2.1, R61.2, SJ3.2, SJ6.2, SJ9.2, U10P.V-, U1A.INH, U1P.GND, U2A.INH, U2P.GND, U3P.VSS, U4P.VSS, U6P.VSS, U7.GND, U7B.VSS, U8.GND1, U8.GND2, U8.GND3, U8.GND4, U8.SD, U8B.!ON/OFF, U8B.GND@PWR, U8B.GNDSIG; no longer C2.2, C6.-, D5.A, D6.A, J1.2, J1.2B, J1.3B, JP1.5, JP1.6, JP10.5, JP2.5, JP2.6, JP3.5, JP3.6, JP4.5, JP4.6, JP5.8, JP6.4, JP9.5, R16.2, R51.1, SJ13.2, SJ19.2, SJ20.2, U1.GND, U10P.VSS, U1B.VSS, U2.GND1, U2.GND2, U2.GND3, U2.GND4, U2.SD, U2B.!ON/OFF, U2B.GND@PWR, U2B.GNDSIG, U3A.INH, U3P.GND, U4A.INH, U4P.GND, U6P.V-, U7P.VSS, U8P.VSS, X1.3, X1.6, X1.7, X2.3, X2.6, X2.7, X3.2, X5.9
- net I2CSCL: now also JP1.1, R62.2; no longer JP6.1, R15.2
- net I2CSDA: now also JP1.2, R63.2; no longer JP6.2, R14.2
- net ILAT: now also U1A.SH/!LD, U2A.SH/!LD; no longer U3A.SH/!LD, U4A.SH/!LD
- net LPOWA: now also SJ7.1, SJ9.1, U14.GND; no longer SJ10.1, SJ12.1, U12.GND
- net LPOWB: now also SJ10.1, SJ12.1, U14.CD+; no longer SJ13.1, SJ9.1, U12.CD+, X8.9
- net MISO: now also JP2.1; no longer JP5.1
- net MISO2: now also SJ13.2, SJ19.2, U2A.QH; no longer SJ1.2, SJ7.2, U3A.QH
- net MISO2_ALT: now also SJ13.1; no longer SJ1.1
- net MOSI: now also R20.1, SJ15.1, SJ17.2, U11A.SER; no longer R4.1, SJ14.2, SJ4.1, U13A.SER
- net N$1: now also R3.1, U11A.QA, U12.I1; no longer R67.1, U13A.QA, U14.I1
- net N$10: now also R6.1, U11A.QD, U12.I4; no longer R64.1, U13A.QD, U14.I4
- net N$100: now also R17.1, U13A.QG, U14.I7; no longer R53.1, U11A.QG, U12.I7
- net N$101: now also Q15.D, U14.O7, X4.7; no longer Q2.D, U12.O7, X8.7
- net N$102: now also R18.1, U13A.QH, U14.I8; no longer R52.1, U11A.QH, U12.I8
- net N$104: now also Q9.G, R11.2; no longer Q8.G, R59.2
- net N$105: now also Q10.G, R12.2; no longer Q7.G, R58.2
- net N$106: now also Q11.G, R13.2; no longer Q6.G, R57.2
- net N$107: now also Q12.G, R14.2; no longer Q5.G, R56.2
- net N$108: now also Q13.G, R15.2; no longer Q4.G, R55.2
- net N$109: now also Q14.G, R16.2; no longer Q3.G, R54.2
- net N$11: now also Q4.D, U12.O4, X5.4; no longer Q13.D, U14.O4, X9.4
- net N$110: now also Q15.G, R17.2; no longer Q2.G, R53.2
- net N$111: now also Q16.G, R18.2; no longer Q1.G, R52.2
- net N$12: now also R7.1, U11A.QE, U12.I5; no longer R63.1, U13A.QE, U14.I5
- net N$13: now also Q5.D, U12.O5, X5.5; no longer Q12.D, U14.O5, X9.5
- net N$14: now also PORTA.9, R37.2, R59.2, RN3G.1, RN4.3, X1.7; no longer JP9.2, R35.2, R48.2, RN3.3, RN4G.1, X5.7
- net N$15: now also PORTA.8, R38.2, R58.2, RN3F.1, RN4.4, X1.6; no longer JP9.3, R36.2, R47.2, RN3.4, RN4F.1, X5.6
- net N$16: now also Q4.G, R6.2; no longer Q13.G, R64.2
- net N$17: now also R8.1, U11A.QF, U12.I6; no longer R62.1, U13A.QF, U14.I6
- net N$18: now also Q6.D, U12.O6, X5.6; no longer Q11.D, U14.O6, X9.6
- net N$19: now also PORTA.4, R41.2, R56.2, RN3D.1, RN4.6, X1.4; no longer JP9.7, R38.2, R45.2, RN3.6, RN4D.1, X5.4
- net N$2: now also Q1.D, U12.O1, X5.1; no longer Q16.D, U14.O1, X9.1
- net N$20: now also PORTA.3, R42.2, R55.2, RN3C.1, RN4.7, X1.3; no longer JP9.8, R39.2, R44.2, RN3.7, RN4C.1, X5.3
- net N$21: now also PORTB.8, R30.2, R50.2, RN1F.1, RN2.4, X2.6; no longer JP8.3, R20.2, R31.2, RN1.4, RN2F.1, X4.6
- net N$22: now also PORTA.1, R44.2, R53.2, RN3A.1, RN4.9, X1.1; no longer JP9.10, R41.2, R42.2, RN3.9, RN4A.1, X5.1
- net N$23: now also R36.1, RN3H.2, U1A.A; no longer R34.1, RN4H.2, U4A.A
- net N$24: now also R37.1, RN3G.2, U1A.B; no longer R35.1, RN4G.2, U4A.B
- net N$25: now also PORTB.10, R28.2, R52.2, RN1H.1, RN2.2, X2.8; no longer JP8.1, R18.2, R33.2, RN1.2, RN2H.1, X4.8
- net N$26: now also PORTB.9, R29.2, R51.2, RN1G.1, RN2.3, X2.7; no longer JP8.2, R19.2, R32.2, RN1.3, RN2G.1, X4.7
- net N$27: now also Q5.G, R7.2; no longer Q12.G, R63.2
- net N$28: now also PORTB.7, R31.2, R49.2, RN1E.1, RN2.5, X2.5; no longer JP8.4, R21.2, R30.2, RN1.5, RN2E.1, X4.5
- net N$29: now also R38.1, RN3F.2, U1A.C; no longer R36.1, RN4F.2, U4A.C
- net N$3: now also R4.1, U11A.QB, U12.I2; no longer R66.1, U13A.QB, U14.I2
- net N$30: now also R39.1, RN3E.2, U1A.D; no longer R37.1, RN4E.2, U4A.D
- net N$31: now also R41.1, RN3D.2, U1A.E; no longer R38.1, RN4D.2, U4A.E
- net N$32: now also R42.1, RN3C.2, U1A.F; no longer R39.1, RN4C.2, U4A.F
- net N$33: now also PORTB.4, R32.2, R48.2, RN1D.1, RN2.6, X2.4; no longer JP8.7, R22.2, R29.2, RN1.6, RN2D.1, X4.4
- net N$34: now also PORTB.3, R33.2, R47.2, RN1C.1, RN2.7, X2.3; no longer JP8.8, R23.2, R28.2, RN1.7, RN2C.1, X4.3
- net N$35: now also PORTB.2, R34.2, R46.2, RN1B.1, RN2.8, X2.2; no longer JP8.9, R24.2, R27.2, RN1.8, RN2B.1, X4.2
- net N$37: now also R43.1, RN3B.2, U1A.G; no longer R40.1, RN4B.2, U4A.G
- net N$38: now also R44.1, RN3A.2, U1A.H; no longer R41.1, RN4A.2, U4A.H
- net N$39: now also R9.1, U11A.QG, U12.I7; no longer R61.1, U13A.QG, U14.I7
- net N$4: now also J1.4, J2.4; no longer D3.A, D4.A, J1.1, J1.1B, X3.1
- net N$40: now also Q7.D, U12.O7, X5.7; no longer Q10.D, U14.O7, X9.7
- net N$41: now also R10.1, U11A.QH, U12.I8; no longer R60.1, U13A.QH, U14.I8
- net N$42: now also Q8.D, U12.O8, X5.8; no longer Q9.D, U14.O8, X9.8
- net N$43: now also Q6.G, R8.2; no longer Q11.G, R62.2
- net N$44: now also R28.1, RN1H.2, U2A.A; no longer R18.1, RN2H.2, U3A.A
- net N$45: now also D4.C, JP4.1; no longer D1.C, JP7.1
- net N$46: now also D4.A, JP4.4; no longer D1.A, JP7.4
- net N$47: now also R29.1, RN1G.2, U2A.B; no longer R19.1, RN2G.2, U3A.B
- net N$48: now also R30.1, RN1F.2, U2A.C; no longer R20.1, RN2F.2, U3A.C
- net N$49: now also R31.1, RN1E.2, U2A.D; no longer R21.1, RN2E.2, U3A.D
- net N$5: now also J1.5, J2.5; no longer JP8.10, R25.2, R26.2, RN1.9, RN2A.1, X4.1
- net N$50: now also R32.1, RN1D.2, U2A.E; no longer R22.1, RN2D.2, U3A.E
- net N$51: now also R33.1, RN1C.2, U2A.F; no longer R23.1, RN2C.2, U3A.F
- net N$52: now also R34.1, RN1B.2, U2A.G; no longer R24.1, RN2B.2, U3A.G
- net N$53: now also R35.1, RN1A.2, U2A.H; no longer R25.1, RN2A.2, U3A.H
- net N$56: now also R11.1, U13A.QA, U14.I1; no longer R59.1, U11A.QA, U12.I1
- net N$57: now also JP4.3, R40.1; no longer JP7.3, R17.1
- net N$6: now also PORTA.10, R36.2, R60.2, RN3H.1, RN4.2, X1.8; no longer JP9.1, R34.2, R49.2, RN3.2, RN4H.1, X5.8
- net N$60: now also SJ14.1; no longer SJ3.1
- net N$65: now also Q7.G, R9.2; no longer Q10.G, R61.2
- net N$7: now also Q2.D, U12.O2, X5.2; no longer Q15.D, U14.O2, X9.2
- net N$75: now also Q16.D, U14.O8, X4.8; no longer Q1.D, U12.O8, X8.8
- net N$78: now also Q1.G, R3.2; no longer Q16.G, R67.2
- net N$79: now also Q2.G, R4.2; no longer Q15.G, R66.2
- net N$8: now also R5.1, U11A.QC, U12.I3; no longer R65.1, U13A.QC, U14.I3
- net N$83: now also PORTA.7, R39.2, R57.2, RN3E.1, RN4.5, X1.5; no longer JP9.4, R37.2, R46.2, RN3.5, RN4E.1, X5.5
- net N$84: now also PORTA.2, R54.2, RN3B.1, RN4.8, X1.2; no longer JP9.9, R40.2, RN3.8, RN4B.1, X5.2
- net N$85: now also Q8.G, R10.2; no longer Q9.G, R60.2
- net N$87: now also Q9.D, U14.O1, X4.1; no longer Q8.D, U12.O1, X8.1
- net N$88: now also Q3.G, R5.2; no longer Q14.G, R65.2
- net N$89: now also R12.1, U13A.QB, U14.I2; no longer R58.1, U11A.QB, U12.I2
- net N$9: now also Q3.D, U12.O3, X5.3; no longer Q14.D, U14.O3, X9.3
- net N$91: now also Q10.D, U14.O2, X4.2; no longer Q7.D, U12.O2, X8.2
- net N$92: now also R13.1, U13A.QC, U14.I3; no longer R57.1, U11A.QC, U12.I3
- net N$93: now also Q11.D, U14.O3, X4.3; no longer Q6.D, U12.O3, X8.3
- net N$94: now also R14.1, U13A.QD, U14.I4; no longer R56.1, U11A.QD, U12.I4
- net N$95: now also Q12.D, U14.O4, X4.4; no longer Q5.D, U12.O4, X8.4
- net N$96: now also R15.1, U13A.QE, U14.I5; no longer R55.1, U11A.QE, U12.I5
- net N$97: now also Q13.D, U14.O5, X4.5; no longer Q4.D, U12.O5, X8.5
- net N$98: now also R16.1, U13A.QF, U14.I6; no longer R54.1, U11A.QF, U12.I6
- net N$99: now also Q14.D, U14.O6, X4.6; no longer Q3.D, U12.O6, X8.6
- net OLAT: now also R21.1; no longer R3.1
- net PWR_POS: now also J1.8, J2.8, R40.2; no longer R17.2, X1.8, X2.8
- net RPOWA: now also SJ1.1, SJ2.1, SJ3.1, U12.GND; no longer SJ15.1, SJ17.1, SJ19.1, U14.GND
- net RPOWB: now also SJ4.1, SJ5.1, SJ6.1, U12.CD+; no longer SJ16.1, SJ18.1, SJ20.1, U14.CD+, X9.9
- net SCK: now also JP2.3, R19.1; no longer JP5.3, R5.1
- net SCK2: now also U1A.CLK, U2A.CLK; no longer SJ2.1, U3A.CLK, U4A.CLK
- net SLNK1: now also SJ17.1, U11A.QH*, U13A.SER; no longer SJ14.1, U11A.SER, U13A.QH*
- net SLNK2: now also SJ16.1, U13A.QH*; no longer SJ5.1, U11A.QH*
- net SLNK3: now also SJ19.1, U1A.QH, U2A.SER; no longer SJ7.1, U3A.SER, U4A.QH
- net SRV1: now also JP5.2, R24.2; no longer JP4.2, R13.2
- net SRV2: now also JP5.1, R25.2; no longer JP4.1, R12.2
- net SRV3: now also JP6.2, R26.2; no longer JP3.2, R11.2
- net SRV4: now also JP6.1, R27.2; no longer JP3.1, R10.2
- net SRV5: now also JP7.2, R64.2, U$1.PF1-PH1; no longer JP2.2, R9.2, U$1.PC12
- net SRV6: now also JP7.1, R65.2; no longer JP2.1, R8.2
- net SRV7: now also JP8.2, R66.2, U$1.PC12; no longer JP1.2, R7.2, U$1.PF1-PH1
- net SRV8: now also JP8.1, R67.2; no longer JP1.1, R6.2
- net SW: now also D1.C, D3.C, U8.VOUT, U8B.OUT; no longer D5.C, D6.C, U2.VOUT, U2B.OUT
- net TDRV1: now also U10D.+IN, U6A.I; no longer U10A.I, U9D.+IN
- net TDRV2: now also U10A.+IN, U6B.I; no longer U10B.I, U9A.+IN
- net TDRV3: now also U10C.+IN, U5B.I; no longer U8B.I, U9C.+IN
- net TDRV4: now also U10B.+IN, U5A.I; no longer U8A.I, U9B.+IN
- net TDRV5: now also U4A.I, U9D.+IN; no longer U6D.+IN, U7A.I
- net TDRV6: now also U4B.I, U9A.+IN; no longer U6A.+IN, U7B.I
- net TDRV7: now also U3B.I, U9C.+IN; no longer U5B.I, U6C.+IN
- net TDRV8: now also U3A.I, U9B.+IN; no longer U5A.I, U6B.+IN
- net TOUT1: now also PORTC.1, U3A.O, U9B.OUT, X3.1; no longer JP10.10, U5A.O, U6B.OUT, X7.1
- net TOUT2: now also PORTC.2, U3B.O, U9C.OUT, X3.2; no longer JP10.9, U5B.O, U6C.OUT, X7.2
- net TOUT3: now also PORTC.3, U4B.O, U9A.OUT, X3.3; no longer JP10.8, U6A.OUT, U7B.O, X7.3
- net TOUT4: now also PORTC.4, U4A.O, U9D.OUT, X3.4; no longer JP10.7, U6D.OUT, U7A.O, X7.4
- net TOUT5: now also PORTC.7, U10B.OUT, U5A.O, X3.5; no longer JP10.4, U8A.O, U9B.OUT, X7.5
- net TOUT6: now also PORTC.8, U10C.OUT, U5B.O, X3.6; no longer JP10.3, U8B.O, U9C.OUT, X7.6
- net TOUT7: now also PORTC.9, U10A.OUT, U6B.O, X3.7; no longer JP10.2, U10B.O, U9A.OUT, X7.7
- net TOUT8: now also PORTC.10, U10D.OUT, U6A.O, X3.8; no longer JP10.1, U10A.O, U9D.OUT, X7.8
- net V+: now also C1.1, C2.+, U8.FB, U8B.FB; no longer C6.+, C7.1, U2.FB, U2B.FB
Other:
- note added: "Alternative population: Output ports D and E are optionally populated. If one output port is needed, populate port D (this sheet) and close SJ17. For options on populating U14, see sheet 6."
- note added: "Alternative population: Populate U9 and U10 to drive stall motor switch machines (e.g. Tortoise). This can also be used for CA or CC LED driving with appropriate external current limit resistors calculated for +15V. Multiple LEDs can be in series, too. Populate U3-U6 with TC4426 or TC4428 to drive high current (up to 1.5A per port) outputs in push-pull mode. Invert the output in software when swi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"
- note added: "Alternative population: This port is optionally populated. If not populated, close SJ17. For U11, may substitute 74HC595N if R19-R21 are populated. For HCT series those resistors are not necessary. For driving LEDs with up to 8 mA current, U12 may be populated with the series resistors for the LEDs directly. If external series resistors are present, the screw terminal can be soldered directly int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"
- note added: "Close S19 if PORTB is not populated."
- note added: "Close for F303RE."
- note added: "Close if 5V-DCDC switcher is not populated. Will use Nucleo's linear regulator from 12V to 5V, which produces a lot of heat; putting any load by external peripherals is not permissible. Might work with lower voltage (e.g. 7V) input power."
- note added: "Close if U11 is missing."
- note added: "If SJ15 is closed, expn port SPI is parallel to onboard shift registers. If SJ15 is open and SJ16 is closed, they get daisy-chained."
- note added: "JP4: Power select jumper Bridge 1-2 and 3-4 in order to be bus powered (take power from OpenLCB bus). Bridge 1-3 and 2-4 in order to supply power to OpenLCB bus. Power plugged in to J3 is needed. Leave open in order to take power from power jack only. Power plugged in to J3 is needed."
- note added: "Populate R24-27 and R64-67 if the servos in use are not compatible with 3V voltage levels. JP7-8 for SRV5-8 shall not be populated if a Nucleo-144 board is used."
- note added: "Populate only one alternative - U8 (SOIC-8) with AP1509 or - U8B (PDIP-8) with LM2574N-5.0 depending on the desired package."
- note added: "Populate only one alternative of U7 (PDIP-8) or U7B (SOIC-8) depending on the package. Example part choice: - MCP2551: R61 optional if slew rate control is needed. SJ18 open. - PCA82C250. R61 is 0 ohm or a slew control resistor. SJ18 open. - MCP2561, ATA6560/62: not recommended. - MCP2562 ATA6561/63: R61 is 0 ohm, SJ18 closed. - SN65HVD1050: R61 is 0 ohm, SJ18 open. - MCP2542FD: R61 is 0 ohm, SJ1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"
- note added: "Through-hole population: - populate RN1, RN3 with parallel resistor network or individual resistors. - populate RN2, RN4 with star resistor network. - DNP R28-R60. SMD population: - populate R28-R60 - DNP RN1-4. Values: - RN1, RN3, R28-R44: 22k-270k. - RN2, RN4, R45-R60: 10k-270k."
- note added: "V+ is 5V power in for the Morpho connector 'E5V' pin. Will supply MCU with power via a linear regulator on the MCU board. The MCU board will connect it to the 5V output pin on the Morpho connector"
- note removed: "Alternative population: Output ports D and E are optionally populated. If one output port is needed, populate port D (this sheet) and close SJ14. For options on populating U12, see sheet 6."
- note removed: "Alternative population: Populate U6 and U9 to drive stall motor switch machines (e.g. Tortoise). This can also be used for CA or CC LED driving with appropriate external current limit resistors calculated for +15V. Multiple LEDs can be in series, too. Populate U5,7,8,10 with TC4426 or TC4427 to drive stall motors with more current needs in push-pull mode. Invert the output in software when switch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"
- note removed: "Alternative population: This port is optionally populated. If not populated, close SJ14. For U13, may substitute 74HC595N if R3-R5 are populated. For HCT series those resistors are not necessary. For driving LEDs with up to 8 mA current, U14 may be populated with the series resistors for the LEDs directly. If external series resistors are present, the screw terminal can be soldered directly into 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"
- note removed: "Close SJ7 if PORTB is not populated."
- note removed: "Close both for F303RE."
- note removed: "Close if 5V-DCDC switcher is not populated. Will use Nucleo's linear regulator from 12V to 5V, which has a strict current limit. Must observe max current consumption of the Nucleo specification, which depends on the input voltage. Putting any load by external peripherals is not recommended. Might work with lower voltage (e.g. 7V) input power."
- note removed: "Close if U13 is missing."
- note removed: "If SJ4 is closed, expn port SPI is parallel to onboard shift registers. If SJ4 is open and SJ5 is closed, they get daisy-chained."
- note removed: "JP7: Power select jumper Bridge 1-2 and 3-4 in order to be bus powered (take power from OpenLCB bus). Bridge 1-3 and 2-4 in order to supply power to OpenLCB bus. Power plugged in to J1 is needed. Leave open in order to take power from power jack only. Power plugged in to J1 is needed."
- note removed: "Populate R6-R13 if the servos in use are not compatible with 3V voltage levels. R6-R13: 5k-20k JP1-2 for SRV5-8 can not be populated if a Nucleo-144 board is used."
- note removed: "Populate only one alternative - U2 (SOIC-8) with AP1509 and L1 with 47 uH inductor, or - U2B (PDIP-8) with LM2574N-5.0 and L1 with 470 uH inductor depending on the desired package."
- note removed: "Populate only one alternative of U1 (PDIP-8) or U1B (SOIC-8) depending on the package. Example part choice: - MCP2551: R16 is 0 ohm or a slew control resistor. SJ18 open. - PCA82C250. R16 is 0 ohm or a slew control resistor. SJ18 open. - MCP2561, ATA6560/62: not recommended. - MCP2562 ATA6561/63: R16 is 0 ohm, SJ18 closed. - SN65HVD1050: R16 is 0 ohm, SJ18 open. - MCP2542FD: R16 is 0 ohm, SJ18 cl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"
- note removed: "R1-R5: 5k-20k"
- note removed: "Through-hole population: - populate RN2, RN4 with parallel resistor network or individual resistors. - populate RN1, RN3 with star resistor network. - do not populate R18-R49. SMD population: - populate R18-R49 - DNP RN1-4. Values: - RN2, RN4, R18-R25, R34-R41: 22k-270k. - RN1, RN3, R26-R33, R42-R49: 10k-270k."
- note removed: "V+ is 5V power in to the Morpho connector 'E5V' pin. Will supply MCU with power via a linear regulator on the MCU board. The MCU board will connect it to the 5V output pin on the Morpho connector"
- moved on the sheet: C1, C10, C11, C3, C4, C5, C7, C8, C9, D2, D3, H1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
