File: eagle/nucleo-io-board/io-board-f-c.sch (EAGLE design)
At the start: 169 parts, among them J1 DCJ0202, P1 9-15V DC, Q1 BSS123, Q10 BSS123, Q11 BSS123, Q12 BSS123, Q13 BSS123, Q14 BSS123, Q15 BSS123, Q16 BSS123, Q2 BSS123, Q3 BSS123, Q4 BSS123, Q5 BSS123, Q6 BSS123, Q7 BSS123, Q8 BSS123, Q9 BSS123, U1 CAN-TXR-PDIP, U10 TC4427, U11 74AHCT595N, U13 74AHCT595N, U1B CAN-TXR-SO8, U2 AP1509-50, U2B LM2574N-5.0, U3 74HC166, U4 74HC166, U5 TC4427, U6 LM324N, U7 TC4427, U8 TC4427, U9 LM324N, X1 RJ45-JACK, X2 RJ45-JACK, X4 M08-SCREW, X5 M09-SCREW, X7 M08-SCREW, X8 PORTD, X9 PORTE

Commit message: More versions of the board design.
Connections:
- net +3V3: now also SJ6.2; no longer SJ6.1
- net CAN_VIO: now also SJ6.1; no longer SJ6.2
Other:
- moved on the sheet: C10, C11, C3, C4, C5, C6, C7, C8, C9, D1, D2, D3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
