File: eagle/nucleo-io-board/io-board-f-e.brd (EAGLE design)
At the start: 100 x 80 mm, 169 parts, among them J1 DCJ0202, P1 9-15V DC, U1 CAN-TXR-PDIP, U10 TC4427, U11 74AHCT595N, U13 74AHCT595N, U1B CAN-TXR-SO8, U2 AP1509-50, U2B LM2574N-5.0, U3 74HC166, U4 74HC166, U5 TC4427, U6 LM324N, U7 TC4427, U8 TC4427, U9 LM324N, X1 RJ45-JACK, X2 RJ45-JACK, X4 M08-SCREW, X5 M09-SCREW, X7 M08-SCREW, X8 PORTD, X9 PORTE

Commit message: More versions of the board design.
Parts:
- moved SJ6 1.53 mm to (38.5, 70.2), flipped to the bottom, turned to 0 degrees
Connections:
- net +3V3: now also SJ6.P$2; no longer SJ6.P$1
- net CAN_VIO: now also SJ6.P$1; no longer SJ6.P$2
Routing:
- net +3V3: track 174.9 -> 171.2 mm
- net CAN_VIO: track 10.9 -> 9.37 mm
- net GND: vias 224 -> 228
Other:
- board text added: "OpenLCB Dev IO Rev. B. 2018-05-11"
- board text removed: "OpenLCB Dev IO Rev. B. 2018-05-06"
