File: eagle/jtag-adapter/jtag-adapter-3-5.brd (EAGLE design)
At the start: 58.4 x 58.4 mm, 40 parts, among them IC1 REG1117, Q1 BSS84, Q2 BSS123, X1 TAGCONNECT, X3 CC3220SF-JTAG-HAT, X5 JTAG-IN, X7 MICRO-USB-B

Commit message: Updates resistor values.
Parts:
- R1, R2, R3, R5, R6, R7: value 270 -> 3k3
- R4: value 330 -> 560
Changed lines of the file:
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@@
 <attribute name="NAME" x="38.227" y="23.368" size="1.016" layer="25" font="vector" ratio="15" rot="R270"/>
 </element>
-<element name="R1" library="rcl" library_urn="urn:adsk.eagle:library:334" package="R0805" package3d_urn="urn:adsk.eagle:package:23553/2" value="270" x="46.99" y="34.29" smashed="yes" rot="R90">
+<element name="R1" library="rcl" library_urn="urn:adsk.eagle:library:334" package="R0805" package3d_urn="urn:adsk.eagle:package:23553/2" value="3k3" x="46.99" y="34.29" smashed="yes" rot="R90">
 <attribute name="NAME" x="54.61" y="33.655" size="1.016" layer="25" font="vector" ratio="15" rot="R90"/>
 </element>
-<element name="R2" library="rcl" library_urn="urn:adsk.eagle:library:334" package="R0805" package3d_urn="urn:adsk.eagle:package:23553/2" value="270" x="49.53" y="34.29" smashed="yes" rot="R90">
+<element name="R2" library="rcl" library_urn="urn:adsk.eagle:library:334" package="R0805" package3d_urn="urn:adsk.eagle:package:23553/2" value="3k3" x="49.53" y="34.29" smashed="yes" rot="R90">
 <attribute name="NAME" x="55.88" y="33.655" size="1.016" layer="25" font="vector" ratio="15" rot="R90"/>
 </element>
-<element name="R3" library="rcl" library_urn="urn:adsk.eagle:library:334" package="R0805" package3d_urn="urn:adsk.eagle:package:23553/2" value="270" x="52.07" y="34.29" smashed="yes" rot="R90">
+<element name="R3" library="rcl" library_urn="urn:adsk.eagle:library:334" package="R0805" package3d_urn="urn:adsk.eagle:package:23553/2" value="3k3" x="52.07" y="34.29" smashed="yes" rot="R90">
 <attribute name="NAME" x="57.15" y="33.655" size="1.016" layer="25" font="vector" ratio="15" rot="R90"/>
 </element>
-<element name="R5" library="rcl" library_urn="urn:adsk.eagle:library:334" package="R0805" package3d_urn="urn:adsk.eagle:package:23553/2" value="270" x="55.88" y="20.32" smashed="yes" rot="R180">
+<element name="R5" library="rcl" library_urn="urn:adsk.eagle:library:334" package="R0805" package3d_urn="urn:adsk.eagle:package:23553/2" value="3k3" x="55.88" y="20.32" smashed="yes" rot="R180">
 <attribute name="NAME" x="56.515" y="29.21" size="1.016" layer="25" font="vector" ratio="15" rot="R180"/>
 </element>
-<element name="R6" library="rcl" library_urn="urn:adsk.eagle:library:334" package="R0805" package3d_urn="urn:adsk.eagle:package:23553/2" value="270" x="55.88" y="22.86" smashed="yes" rot="R180">
+<element name="R6" library="rcl" library_urn="urn:adsk.eagle:library:334" package="R0805" package3d_urn="urn:adsk.eagle:package:23553/2" value="3k3" x="55.88" y="22.86" smashed="yes" rot="R180">
 <attribute name="NAME" x="56.515" y="30.48" size="1.016" layer="25" font="vector" ratio="15" rot="R180"/>
 </element>
-<element name="R7" library="rcl" library_urn="urn:adsk.eagle:library:334" package="R0805" package3d_urn="urn:adsk.eagle:package:23553/2" value="270" x="55.88" y="25.4" smashed="yes" rot="R180">
+<element name="R7" library="rcl" library_urn="urn:adsk.eagle:library:334" package="R0805" package3d_urn="urn:adsk.eagle:package:23553/2" value="3k3" x="55.88" y="25.4" smashed="yes" rot="R180">
 <attribute name="NAME" x="56.515" y="31.75" size="1.016" layer="25" font="vector" ratio="15" rot="R180"/>
 </element>
@@
 <attribute name="VALUE" x="33.02" y="17.018" size="1.016" layer="27" font="vector" ratio="15" rot="R180"/>
 </element>
-<element name="R4" library="rcl" library_urn="urn:adsk.eagle:library:334" package="R0805" package3d_urn="urn:adsk.eagle:package:23553/2" value="330" x="26.67" y="33.02" smashed="yes" rot="R270">
+<element name="R4" library="rcl" library_urn="urn:adsk.eagle:library:334" package="R0805" package3d_urn="urn:adsk.eagle:package:23553/2" value="560" x="26.67" y="33.02" smashed="yes" rot="R270">
 <attribute name="NAME" x="25.908" y="30.226" size="1.016" layer="25" font="vector" ratio="15"/>
 </element>
